Commit message: Fix for BlueROV in HoloOcean

File: coug_description/urdf/bluerov2_holoocean/bluerov2_holoocean.urdf.xacro (robot description, xacro)
@@ -45,5 +45,5 @@
     <parent link="com_link"/>
     <child link="dvl_link"/>
-    <origin xyz="0 0.1 -0.1" rpy="0 0 0"/>
+    <origin xyz="0 -0.1 -0.1" rpy="0 0 0"/>
   </joint>
   <link name="dvl_link"/>
