Commit message: Better AQUA-SLAM URDFs

File: coug_description/urdf/aquaslam.urdf.xacro (robot description, xacro)
@@ -23,5 +23,5 @@
     <parent link="base_link"/>
     <child link="imu_link"/>
-    <origin xyz="-0.211573 -0.054312 -0.098612" rpy="-1.548854 0.012316 3.122423"/>
+    <origin xyz="-0.214252 -0.051701 -0.094119" rpy="-1.581110 -0.017474 3.125071"/>
   </joint>
   <!-- Depth Link -->
@@ -30,5 +30,5 @@
     <parent link="base_link"/>
     <child link="depth_link"/>
-    <origin xyz="-0.211573 -0.054312 -0.098612" rpy="0 0 0"/>
+    <origin xyz="-0.214252 -0.051701 -0.094119" rpy="0 0 0"/>
   </joint>
   <!-- DVL Link -->
@@ -37,5 +37,5 @@
     <parent link="base_link"/>
     <child link="dvl_link"/>
-    <origin xyz="-0.132345 0.032086 -0.240100" rpy="${pi} 0 0"/>
+    <origin xyz="-0.139380 0.039519 -0.234959" rpy="-3.108800 0.029221 0.003060"/>
   </joint>
 </robot>

File: coug_description/urdf/aquaslam_wt.urdf.xacro (robot description, xacro)
@@ -23,5 +23,5 @@
     <parent link="base_link"/>
     <child link="imu_link"/>
-    <origin xyz="-0.211573 -0.054312 -0.098612" rpy="-1.548854 0.012316 3.122423"/>
+    <origin xyz="-0.229713 -0.064365 -0.141380" rpy="-2.622725 -1.474140 -2.101867"/>
   </joint>
   <!-- Depth Link -->
@@ -30,5 +30,5 @@
     <parent link="base_link"/>
     <child link="depth_link"/>
-    <origin xyz="-0.211573 -0.054312 -0.098612" rpy="0 0 0"/>
+    <origin xyz="-0.229713 -0.064365 -0.141380" rpy="0 0 0"/>
   </joint>
   <!-- DVL Link -->
@@ -37,5 +37,5 @@
     <parent link="base_link"/>
     <child link="dvl_link"/>
-    <origin xyz="-0.132345 0.032086 -0.240100" rpy="${pi} 0 0"/>
+    <origin xyz="-0.153627 0.011795 -0.195926" rpy="-3.120647 -0.023655 0.052659"/>
   </joint>
 </robot>
