Commit message: Add gps link to holoocean URDFs

File: coug_description/urdf/bluerov2_holoocean.urdf.xacro (robot description, xacro)
@@ -27,4 +27,16 @@
   </joint>
   <link name="com_link"/>
+  <joint name="gps_joint" type="fixed">
+    <parent link="base_link"/>
+    <child link="gps_link"/>
+    <origin xyz="0 0 0" rpy="0 0 0"/>
+  </joint>
+  <link name="gps_link"/>
+  <joint name="modem_joint" type="fixed">
+    <parent link="com_link"/>
+    <child link="modem_link"/>
+    <origin xyz="0 0 0" rpy="0 0 0"/>
+  </joint>
+  <link name="modem_link"/>
   <!-- IMUSocket -->
   <joint name="imu_joint" type="fixed">
@@ -62,11 +74,5 @@
   </joint>
   <link name="sonar_link"/>
-  <!-- Fixes for matching CougUV URDF -->
-  <joint name="modem_joint" type="fixed">
-    <parent link="com_link"/>
-    <child link="modem_link"/>
-    <origin xyz="0 0 0" rpy="0 0 0"/>
-  </joint>
-  <link name="modem_link"/>
+  <!-- Fix for matching CougUV URDF -->
   <joint name="truth_joint" type="fixed">
     <parent link="base_link"/>

File: coug_description/urdf/couguv_holoocean.urdf.xacro (robot description, xacro)
@@ -113,4 +113,10 @@
   </joint>
   <link name="com_link"/>
+  <joint name="gps_joint" type="fixed">
+    <parent link="base_link"/>
+    <child link="gps_link"/>
+    <origin xyz="0 0 0" rpy="0 0 0"/>
+  </joint>
+  <link name="gps_link"/>
   <!-- IMUSocket -->
   <joint name="imu_joint" type="fixed">

Commit message: Add CougUV URDF

File: coug_description/urdf/bluerov2_holoocean.urdf.xacro (robot description, xacro)
@@ -28,5 +28,5 @@
   <link name="com_link"/>
   <joint name="gps_joint" type="fixed">
-    <parent link="base_link"/>
+    <parent link="com_link"/>
     <child link="gps_link"/>
     <origin xyz="0 0 0" rpy="0 0 0"/>
