Commit message: Added WAM-V lever arms

File: coug_description/urdf/bluerov2_holoocean.urdf.xacro (robot description, xacro)
@@ -97,5 +97,5 @@
   </joint>
   <link name="sonar_link"/>
-  <!-- Fix for matching CougUV URDF -->
+  <!-- Fix for HoloOcean GT offset bug -->
   <joint name="truth_joint" type="fixed">
     <parent link="base_link"/>

File: coug_description/urdf/couguv_holoocean.urdf.xacro (robot description, xacro)
@@ -147,5 +147,5 @@
   </joint>
   <link name="dvl_link"/>
-  <!-- Fix for HoloOcean COM offset bug -->
+  <!-- Fix for HoloOcean GT offset bug -->
   <joint name="truth_joint" type="fixed">
     <parent link="base_link"/>

File: coug_description/urdf/wamv_holoocean.urdf.xacro (robot description, xacro)
@@ -48,26 +48,7 @@
   <xacro:engine prefix="right" y="-1.027135"/>
   <!-- NOTE: These are exact HoloOcean socket locations as of 2.0.1 -->
-  <!-- Platform -->
-  <joint name="com_joint" type="fixed">
+  <!-- Payload -->
+  <joint name="depth_joint" type="fixed">
     <parent link="base_link"/>
-    <child link="com_link"/>
-    <origin xyz="0 0 0" rpy="0 0 0"/>
-  </joint>
-  <link name="com_link"/>
-  <joint name="gps_joint" type="fixed">
-    <parent link="com_link"/>
-    <child link="gps_link"/>
-    <origin xyz="0 0 0" rpy="0 0 0"/>
-  </joint>
-  <link name="gps_link"/>
-  <joint name="imu_joint" type="fixed">
-    <parent link="com_link"/>
-    <child link="imu_link"/>
-    <origin xyz="0 0 0" rpy="0 0 0"/>
-  </joint>
-  <link name="imu_link"/>
-  <!-- Payload -->
-   <joint name="depth_joint" type="fixed">
-    <parent link="com_link"/>
     <child link="depth_link"/>
     <origin xyz="0 0 0" rpy="0 ${pi/2} 0"/>
@@ -75,5 +56,5 @@
   <link name="depth_link"/>
   <joint name="dvl_joint" type="fixed">
-    <parent link="com_link"/>
+    <parent link="base_link"/>
     <child link="dvl_link"/>
     <origin xyz="0 0 0" rpy="0 ${pi/2} 0"/>
@@ -81,14 +62,27 @@
   <link name="dvl_link"/>
   <joint name="modem_joint" type="fixed">
-    <parent link="com_link"/>
+    <parent link="base_link"/>
     <child link="modem_link"/>
     <origin xyz="0 0 0" rpy="0 ${pi/2} 0"/>
   </joint>
   <link name="modem_link"/>
-  <!-- Fix for matching CougUV URDF -->
+  <!-- Platform -->
+  <joint name="gps_joint" type="fixed">
+    <parent link="base_link"/>
+    <child link="gps_link"/>
+    <origin xyz="0.55 0 1.3" rpy="0 0 0"/>
+  </joint>
+  <link name="gps_link"/>
+  <joint name="imu_joint" type="fixed">
+    <parent link="base_link"/>
+    <child link="imu_link"/>
+    <origin xyz="0.55 0 1.3" rpy="0 0 0"/>
+  </joint>
+  <link name="imu_link"/>
+  <!-- Fix for HoloOcean GT offset bug -->
   <joint name="truth_joint" type="fixed">
     <parent link="base_link"/>
     <child link="truth_link"/>
-    <origin xyz="0 0 0" rpy="0 0 0"/>
+    <origin xyz="-0.55 0 0" rpy="0 0 0"/>
   </joint>
   <link name="truth_link"/>

Commit message: Add 2.4.0 sockets

File: coug_description/urdf/bluerov2_holoocean.urdf.xacro (robot description, xacro)
@@ -42,5 +42,5 @@
   <xacro:thruster name="thruster7" xyz="-0.118 -0.215 0.064" rpy="0 0 0" mesh="t200_cw_prop.dae"  vis_rpy="1.571 0 1.571"/>
   <xacro:thruster name="thruster8" xyz="-0.118 0.215 0.064"  rpy="0 0 0" mesh="t200_ccw_prop.dae" vis_rpy="-1.571 0 1.571"/>
-  <!-- NOTE: These are exact HoloOcean socket locations as of 2.0.1 -->
+  <!-- NOTE: These are exact HoloOcean socket locations as of 2.4.0 -->
   <!-- COM -->
   <joint name="com_joint" type="fixed">

File: coug_description/urdf/couguv_holoocean.urdf.xacro (robot description, xacro)
@@ -105,5 +105,5 @@
   <xacro:fin_macro prefix="left"  rpy="${pi*2/3} 0 0"/>
   <xacro:fin_macro prefix="right" rpy="${-pi*2/3} 0 0"/>
-  <!-- NOTE: These are exact HoloOcean socket locations as of 2.0.1 -->
+  <!-- NOTE: These are exact HoloOcean socket locations as of 2.4.0 -->
   <!-- COM -->
   <joint name="com_joint" type="fixed">
@@ -123,5 +123,5 @@
     <parent link="com_link"/>
     <child link="imu_link"/>
-    <origin xyz="0.475 0 -0.035" rpy="${pi} 0 0"/>
+    <origin xyz="0.504 0 -0.053" rpy="0 0 0"/>
   </joint>
   <link name="imu_link"/>
@@ -130,5 +130,5 @@
     <parent link="com_link"/>
     <child link="depth_link"/>
-    <origin xyz="0.15 0 0.018" rpy="0 0 0"/>
+    <origin xyz="0.162 0 0" rpy="0 0 0"/>
   </joint>
   <link name="depth_link"/>
@@ -137,5 +137,5 @@
     <parent link="com_link"/>
     <child link="modem_link"/>
-    <origin xyz="0.35 0 -0.086" rpy="0 0 0"/>
+    <origin xyz="0.3785 0 -0.0985" rpy="0 0 0"/>
   </joint>
   <link name="modem_link"/>
@@ -144,12 +144,19 @@
     <parent link="com_link"/>
     <child link="dvl_link"/>
-    <origin xyz="0.475 0 -0.035" rpy="${pi} 0 0"/>
+    <origin xyz="0.504 0 -0.053" rpy="0 0 0"/>
   </joint>
   <link name="dvl_link"/>
+  <!-- CameraSocket -->
+  <joint name="camera_joint" type="fixed">
+    <parent link="com_link"/>
+    <child link="camera_link"/>
+    <origin xyz="0.1 0 0" rpy="0 ${pi/2} 0"/>
+  </joint>
+  <link name="camera_link"/>
   <!-- Fix for HoloOcean GT offset bug -->
   <joint name="truth_joint" type="fixed">
     <parent link="base_link"/>
     <child link="truth_link"/>
-    <origin xyz="-0.1 0 -0.1" rpy="0 0 0"/>
+    <origin xyz="0 0 0" rpy="0 0 0"/>
   </joint>
   <link name="truth_link"/>

File: coug_description/urdf/wamv_holoocean.urdf.xacro (robot description, xacro)
@@ -47,5 +47,5 @@
   <xacro:engine prefix="left"  y="1.027135"/>
   <xacro:engine prefix="right" y="-1.027135"/>
-  <!-- NOTE: These are exact HoloOcean socket locations as of 2.0.1 -->
+  <!-- NOTE: These are exact HoloOcean socket locations as of 2.4.0 -->
   <!-- Payload -->
   <joint name="depth_joint" type="fixed">

Commit message: Fixed robot_localization gravity mishandling bug

File: coug_description/urdf/bluerov2_holoocean.urdf.xacro (robot description, xacro)
@@ -66,5 +66,6 @@
     <parent link="com_link"/>
     <child link="imu_link"/>
-    <origin xyz="0.11 0 0.065" rpy="${pi} 0 0"/>
+    <!-- IMU pitched 180 deg in socket due to robot_localization gravity mishandling bug -->
+    <origin xyz="0.11 0 0.065" rpy="0 0 0"/>
   </joint>
   <link name="imu_link"/>

File: coug_description/urdf/couguv_holoocean.urdf.xacro (robot description, xacro)
@@ -123,5 +123,6 @@
     <parent link="com_link"/>
     <child link="imu_link"/>
-    <origin xyz="0.475 0 -0.035" rpy="${pi} 0 0"/>
+    <!-- IMU pitched 180 deg in socket due to robot_localization gravity mishandling bug -->
+    <origin xyz="0.475 0 -0.035" rpy="0 0 0"/>
   </joint>
   <link name="imu_link"/>

Commit message: Remove old truth link correction

File: coug_description/urdf/bluerov2_holoocean.urdf.xacro (robot description, xacro)
@@ -107,11 +107,4 @@
   </joint>
   <link name="sonar_link" />
-  <!-- Fix for HoloOcean GT offset bug -->
-  <joint name="truth_joint" type="fixed">
-    <parent link="base_link" />
-    <child link="truth_link" />
-    <origin xyz="0 0 0" rpy="0 0 0" />
-  </joint>
-  <link name="truth_link" />
   <!-- Configured stereo camera poses -->
   <!-- IMPORTANT! In HoloOcean, cameras look along X, with Z up and Y left -->

File: coug_description/urdf/couguv_holoocean.urdf.xacro (robot description, xacro)
@@ -179,10 +179,3 @@
   </joint>
   <link name="camera_link" />
-  <!-- Fix for HoloOcean GT offset bug -->
-  <joint name="truth_joint" type="fixed">
-    <parent link="base_link" />
-    <child link="truth_link" />
-    <origin xyz="0 0 0" rpy="0 0 0" />
-  </joint>
-  <link name="truth_link" />
 </robot>

File: coug_description/urdf/wamv_holoocean.urdf.xacro (robot description, xacro)
@@ -80,10 +80,3 @@
   </joint>
   <link name="imu_link" />
-  <!-- Fix for HoloOcean GT offset bug -->
-  <joint name="truth_joint" type="fixed">
-    <parent link="base_link" />
-    <child link="truth_link" />
-    <origin xyz="0 0 0" rpy="0 0 0" />
-  </joint>
-  <link name="truth_link" />
 </robot>

Commit message: Add depth camera link to BlueROV2

File: coug_description/urdf/bluerov2_holoocean.urdf.xacro (robot description, xacro)
@@ -129,3 +129,10 @@
   </joint>
   <link name="back_stereo_link" />
+  <!-- Configured depth camera pose (optical frame) -->
+  <joint name="depth_camera_joint" type="fixed">
+    <parent link="dvl_link" />
+    <child link="depth_camera_link" />
+    <origin xyz="0 0 0" rpy="${pi} 0 ${-pi/2}" />
+  </joint>
+  <link name="depth_camera_link" />
 </robot>

Commit message: Better camera frame handling

File: coug_description/urdf/bluerov2_holoocean.urdf.xacro (robot description, xacro)
@@ -116,23 +116,41 @@
   </joint>
   <link name="sonar_link" />
-  <!-- Configured stereo camera poses (optical frame) -->
+  <!-- Configured stereo camera poses -->
   <joint name="front_stereo_joint" type="fixed">
     <parent link="dvl_link" />
     <child link="front_stereo_link" />
-    <origin xyz="0.1 0 0" rpy="${pi} 0 ${-pi/2}" />
+    <origin xyz="0.1 0 0" rpy="0 ${pi/2} 0" />
   </joint>
   <link name="front_stereo_link" />
+  <joint name="front_stereo_optical_joint" type="fixed">
+    <parent link="front_stereo_link" />
+    <child link="front_stereo_optical_link" />
+    <origin xyz="0 0 0" rpy="${-pi/2} 0 ${-pi/2}" />
+  </joint>
+  <link name="front_stereo_optical_link" />
   <joint name="back_stereo_joint" type="fixed">
     <parent link="dvl_link" />
     <child link="back_stereo_link" />
-    <origin xyz="-0.1 0 0" rpy="${pi} 0 ${-pi/2}" />
+    <origin xyz="-0.1 0 0" rpy="0 ${pi/2} 0" />
   </joint>
   <link name="back_stereo_link" />
-  <!-- Configured depth camera pose (optical frame) -->
+  <joint name="back_stereo_optical_joint" type="fixed">
+    <parent link="back_stereo_link" />
+    <child link="back_stereo_optical_link" />
+    <origin xyz="0 0 0" rpy="${-pi/2} 0 ${-pi/2}" />
+  </joint>
+  <link name="back_stereo_optical_link" />
+  <!-- Configured depth camera pose -->
   <joint name="depth_camera_joint" type="fixed">
     <parent link="dvl_link" />
     <child link="depth_camera_link" />
-    <origin xyz="0 0 0" rpy="${pi} 0 ${-pi/2}" />
+    <origin xyz="0 0 0" rpy="0 ${pi/2} 0" />
   </joint>
   <link name="depth_camera_link" />
+  <joint name="depth_camera_optical_joint" type="fixed">
+    <parent link="depth_camera_link" />
+    <child link="depth_camera_optical_link" />
+    <origin xyz="0 0 0" rpy="${-pi/2} 0 ${-pi/2}" />
+  </joint>
+  <link name="depth_camera_optical_link" />
 </robot>

File: coug_description/urdf/couguv_holoocean.urdf.xacro (robot description, xacro)
@@ -188,10 +188,16 @@
   </joint>
   <link name="camera_link" />
-  <!-- Configured depth camera pose (optical frame) -->
+  <!-- Configured depth camera pose -->
   <joint name="depth_camera_joint" type="fixed">
     <parent link="dvl_link" />
     <child link="depth_camera_link" />
-    <origin xyz="0 0 0" rpy="${pi} 0 ${-pi/2}" />
+    <origin xyz="0 0 0" rpy="0 ${pi/2} 0" />
   </joint>
   <link name="depth_camera_link" />
+  <joint name="depth_camera_optical_joint" type="fixed">
+    <parent link="depth_camera_link" />
+    <child link="depth_camera_optical_link" />
+    <origin xyz="0 0 0" rpy="${-pi/2} 0 ${-pi/2}" />
+  </joint>
+  <link name="depth_camera_optical_link" />
 </robot>

Commit message: Add WAM-V depth camera

File: coug_description/urdf/bluerov2_holoocean.urdf.xacro (robot description, xacro)
@@ -100,19 +100,4 @@
   <xacro:dvl_beam prefix="beam2" yaw="${radians(180)}" />
   <xacro:dvl_beam prefix="beam3" yaw="${radians(-90)}" />
-  <!-- CameraSocket -->
-  <joint name="camera_joint" type="fixed">
-    <parent link="com_link" />
-    <child link="camera_link" />
-    <origin xyz="0.21 0 0.06" rpy="0 0 0" />
-  </joint>
-  <link name="camera_link" />
-  <!-- SonarSocket -->
-  <joint name="sonar_joint" type="fixed">
-    <parent link="com_link" />
-    <child link="sonar_link" />
-    <origin xyz="0.15 0 0.14" rpy="0 0 0" />
-  </joint>
-  <link name="sonar_link" />
-  <!-- Configured stereo camera poses -->
   <joint name="front_stereo_joint" type="fixed">
     <parent link="dvl_link" />
@@ -139,5 +124,4 @@
   </joint>
   <link name="back_stereo_optical_link" />
-  <!-- Configured depth camera pose -->
   <joint name="depth_camera_joint" type="fixed">
     <parent link="dvl_link" />
@@ -152,3 +136,17 @@
   </joint>
   <link name="depth_camera_optical_link" />
+  <!-- CameraSocket -->
+  <joint name="camera_joint" type="fixed">
+    <parent link="com_link" />
+    <child link="camera_link" />
+    <origin xyz="0.21 0 0.06" rpy="0 0 0" />
+  </joint>
+  <link name="camera_link" />
+  <!-- SonarSocket -->
+  <joint name="sonar_joint" type="fixed">
+    <parent link="com_link" />
+    <child link="sonar_link" />
+    <origin xyz="0.15 0 0.14" rpy="0 0 0" />
+  </joint>
+  <link name="sonar_link" />
 </robot>

File: coug_description/urdf/couguv_holoocean.urdf.xacro (robot description, xacro)
@@ -187,20 +187,4 @@
   <xacro:dvl_beam prefix="beam2" yaw="${radians(180)}" />
   <xacro:dvl_beam prefix="beam3" yaw="${radians(-90)}" />
-  <!-- AcousticModemSocket -->
-  <joint name="modem_joint" type="fixed">
-    <parent link="com_link" />
-    <child link="modem_link" />
-    <!-- Sensor FLU frame; FRD data converted upstream -->
-    <origin xyz="0.3785 0 -0.0985" rpy="0 0 0" />
-  </joint>
-  <link name="modem_link" />
-  <!-- CameraSocket -->
-  <joint name="camera_joint" type="fixed">
-    <parent link="com_link" />
-    <child link="camera_link" />
-    <origin xyz="0.1 0 0" rpy="0 ${radians(90)} 0" />
-  </joint>
-  <link name="camera_link" />
-  <!-- Configured depth camera pose -->
   <joint name="depth_camera_joint" type="fixed">
     <parent link="dvl_link" />
@@ -215,3 +199,18 @@
   </joint>
   <link name="depth_camera_optical_link" />
+  <!-- AcousticModemSocket -->
+  <joint name="modem_joint" type="fixed">
+    <parent link="com_link" />
+    <child link="modem_link" />
+    <!-- Sensor FLU frame; FRD data converted upstream -->
+    <origin xyz="0.3785 0 -0.0985" rpy="0 0 0" />
+  </joint>
+  <link name="modem_link" />
+  <!-- CameraSocket -->
+  <joint name="camera_joint" type="fixed">
+    <parent link="com_link" />
+    <child link="camera_link" />
+    <origin xyz="0.1 0 0" rpy="0 ${radians(90)} 0" />
+  </joint>
+  <link name="camera_link" />
 </robot>

File: coug_description/urdf/wamv_holoocean.urdf.xacro (robot description, xacro)
@@ -88,3 +88,15 @@
   </joint>
   <link name="imu_link" />
+  <joint name="depth_camera_joint" type="fixed">
+    <parent link="base_link" />
+    <child link="depth_camera_link" />
+    <origin xyz="2.0 0 2.0" rpy="0 ${radians(15)} 0" />
+  </joint>
+  <link name="depth_camera_link" />
+  <joint name="depth_camera_optical_joint" type="fixed">
+    <parent link="depth_camera_link" />
+    <child link="depth_camera_optical_link" />
+    <origin xyz="0 0 0" rpy="${radians(-90)} 0 ${radians(-90)}" />
+  </joint>
+  <link name="depth_camera_optical_link" />
 </robot>
