Commit message: Better URDF files

File: coug_description/urdf/bluerov2_holoocean.urdf.xacro (robot description, xacro)
@@ -12,5 +12,5 @@
  limitations under the License.
 -->
-<robot name="bluerov2" xmlns:xacro="http://www.ros.org/wiki/xacro">
+<robot name="bluerov2_holoocean" xmlns:xacro="http://www.ros.org/wiki/xacro">
   <xacro:arg name="tf_prefix" default="" />
   <xacro:property name="tf_prefix" value="$(arg tf_prefix)" />

File: coug_description/urdf/couguv.urdf.xacro (robot description, xacro)
@@ -69,17 +69,4 @@
     </visual>
   </xacro:macro>
-  <xacro:macro name="fin" params="prefix rpy">
-    <joint name="${prefix}_fin_joint" type="revolute">
-      <parent link="${tf_prefix}base_link" />
-      <child link="${tf_prefix}${prefix}_fin_link" />
-      <origin xyz="${-fin_xoff} 0 0" rpy="${rpy}" />
-      <axis xyz="0 0 1" />
-      <limit lower="${radians(-45)}" upper="${radians(45)}" effort="10.0" velocity="1.0" />
-    </joint>
-    <link name="${tf_prefix}${prefix}_fin_link">
-      <xacro:add_box color="White" xyz="${-fin_length/2} 0 ${base_radius+fin_height/2}" rpy="0 0 0"
-        x="${fin_length}" y="${fin_width}" z="${fin_height}" />
-    </link>
-  </xacro:macro>
   <!-- Body -->
   <link name="${tf_prefix}base_link" />
@@ -147,4 +134,17 @@
   </link>
   <!-- Fins -->
+  <xacro:macro name="fin" params="prefix rpy">
+    <joint name="${prefix}_fin_joint" type="revolute">
+      <parent link="${tf_prefix}base_link" />
+      <child link="${tf_prefix}${prefix}_fin_link" />
+      <origin xyz="${-fin_xoff} 0 0" rpy="${rpy}" />
+      <axis xyz="0 0 1" />
+      <limit lower="${radians(-45)}" upper="${radians(45)}" effort="10.0" velocity="1.0" />
+    </joint>
+    <link name="${tf_prefix}${prefix}_fin_link">
+      <xacro:add_box color="White" xyz="${-fin_length/2} 0 ${base_radius+fin_height/2}" rpy="0 0 0"
+        x="${fin_length}" y="${fin_width}" z="${fin_height}" />
+    </link>
+  </xacro:macro>
   <xacro:fin prefix="top" rpy="0 0 0" />
   <xacro:fin prefix="left" rpy="${radians(120)} 0 0" />

File: coug_description/urdf/couguv_holoocean.urdf.xacro (robot description, xacro)
@@ -12,5 +12,5 @@
  limitations under the License.
 -->
-<robot name="couguv" xmlns:xacro="http://www.ros.org/wiki/xacro">
+<robot name="couguv_holoocean" xmlns:xacro="http://www.ros.org/wiki/xacro">
   <xacro:arg name="tf_prefix" default="" />
   <xacro:property name="tf_prefix" value="$(arg tf_prefix)" />
@@ -69,4 +69,71 @@
     </visual>
   </xacro:macro>
+  <!-- Body -->
+  <link name="${tf_prefix}base_link" />
+  <joint name="clear_body_joint" type="fixed">
+    <parent link="${tf_prefix}base_link" />
+    <child link="${tf_prefix}clear_body_link" />
+    <origin xyz="0 0 0" rpy="0 0 0" />
+  </joint>
+  <link name="${tf_prefix}clear_body_link">
+    <xacro:add_cylinder color="Acrylic" xyz="0 0 0" rpy="0 ${radians(90)} 0"
+      radius="${base_radius}" length="${enclosure_length}" />
+  </link>
+  <joint name="front_body_joint" type="fixed">
+    <parent link="${tf_prefix}base_link" />
+    <child link="${tf_prefix}front_body_link" />
+    <origin xyz="${(base_length - 2*base_radius - enclosure_length)/4 + enclosure_length/2} 0 0" rpy="0 0 0" />
+  </joint>
+  <link name="${tf_prefix}front_body_link">
+    <xacro:add_cylinder color="Blue" xyz="0 0 0" rpy="0 ${radians(90)} 0" radius="${base_radius}"
+      length="${(base_length - 2*base_radius - enclosure_length)/2}" />
+  </link>
+  <joint name="back_body_joint" type="fixed">
+    <parent link="${tf_prefix}base_link" />
+    <child link="${tf_prefix}back_body_link" />
+    <origin xyz="${-((base_length - 2*base_radius - enclosure_length)/4 + enclosure_length/2)} 0 0" rpy="0 0 0" />
+  </joint>
+  <link name="${tf_prefix}back_body_link">
+    <xacro:add_cylinder color="Blue" xyz="0 0 0" rpy="0 ${radians(90)} 0" radius="${base_radius}"
+      length="${(base_length - 2*base_radius - enclosure_length)/2}" />
+  </link>
+  <!-- Handle -->
+  <joint name="handle_joint" type="fixed">
+    <parent link="${tf_prefix}base_link" />
+    <child link="${tf_prefix}handle_link" />
+    <origin xyz="0 0 ${base_radius + handle_height/2}" rpy="0 0 0" />
+  </joint>
+  <link name="${tf_prefix}handle_link">
+    <xacro:add_box color="White" xyz="0 0 0" rpy="0 0 0" x="${handle_length}" y="${handle_width}" z="${handle_height}" />
+  </link>
+  <!-- Tray -->
+  <joint name="tray_joint" type="fixed">
+    <parent link="${tf_prefix}base_link" />
+    <child link="${tf_prefix}tray_link" />
+    <origin xyz="0 0 ${-(base_radius + tray_height/2)}" rpy="0 0 0" />
+  </joint>
+  <link name="${tf_prefix}tray_link">
+    <xacro:add_box color="White" xyz="0 0 0" rpy="0 0 0" x="${tray_length}" y="${tray_width}" z="${tray_height}" />
+  </link>
+  <!-- Hull -->
+  <joint name="hull_joint" type="fixed">
+    <parent link="${tf_prefix}base_link" />
+    <child link="${tf_prefix}hull_link" />
+    <origin xyz="${(base_length-2*base_radius)/2} 0 0" rpy="0 0 0" />
+  </joint>
+  <link name="${tf_prefix}hull_link">
+    <xacro:add_sphere color="Blue" xyz="0 0 0" rpy="0 0 0" radius="${base_radius}" />
+  </link>
+  <!-- Thruster -->
+  <joint name="thruster_joint" type="fixed">
+    <parent link="${tf_prefix}base_link" />
+    <child link="${tf_prefix}thruster_link" />
+    <origin xyz="${-(base_length-2*base_radius)/2} 0 0" rpy="0 0 0" />
+  </joint>
+  <link name="${tf_prefix}thruster_link">
+    <xacro:add_cylinder color="Gray" xyz="0 0 0" rpy="0 ${radians(90)} 0"
+      radius="${base_radius*0.9}" length="${2*base_radius}" />
+  </link>
+  <!-- Fins -->
   <xacro:macro name="fin" params="prefix rpy">
     <joint name="${prefix}_fin_joint" type="revolute">
@@ -82,71 +149,4 @@
     </link>
   </xacro:macro>
-  <!-- Body -->
-  <link name="${tf_prefix}base_link" />
-  <joint name="clear_body_joint" type="fixed">
-    <parent link="${tf_prefix}base_link" />
-    <child link="${tf_prefix}clear_body_link" />
-    <origin xyz="0 0 0" rpy="0 0 0" />
-  </joint>
-  <link name="${tf_prefix}clear_body_link">
-    <xacro:add_cylinder color="Acrylic" xyz="0 0 0" rpy="0 ${radians(90)} 0"
-      radius="${base_radius}" length="${enclosure_length}" />
-  </link>
-  <joint name="front_body_joint" type="fixed">
-    <parent link="${tf_prefix}base_link" />
-    <child link="${tf_prefix}front_body_link" />
-    <origin xyz="${(base_length - 2*base_radius - enclosure_length)/4 + enclosure_length/2} 0 0" rpy="0 0 0" />
-  </joint>
-  <link name="${tf_prefix}front_body_link">
-    <xacro:add_cylinder color="Blue" xyz="0 0 0" rpy="0 ${radians(90)} 0" radius="${base_radius}"
-      length="${(base_length - 2*base_radius - enclosure_length)/2}" />
-  </link>
-  <joint name="back_body_joint" type="fixed">
-    <parent link="${tf_prefix}base_link" />
-    <child link="${tf_prefix}back_body_link" />
-    <origin xyz="${-((base_length - 2*base_radius - enclosure_length)/4 + enclosure_length/2)} 0 0" rpy="0 0 0" />
-  </joint>
-  <link name="${tf_prefix}back_body_link">
-    <xacro:add_cylinder color="Blue" xyz="0 0 0" rpy="0 ${radians(90)} 0" radius="${base_radius}"
-      length="${(base_length - 2*base_radius - enclosure_length)/2}" />
-  </link>
-  <!-- Handle -->
-  <joint name="handle_joint" type="fixed">
-    <parent link="${tf_prefix}base_link" />
-    <child link="${tf_prefix}handle_link" />
-    <origin xyz="0 0 ${base_radius + handle_height/2}" rpy="0 0 0" />
-  </joint>
-  <link name="${tf_prefix}handle_link">
-    <xacro:add_box color="White" xyz="0 0 0" rpy="0 0 0" x="${handle_length}" y="${handle_width}" z="${handle_height}" />
-  </link>
-  <!-- Tray -->
-  <joint name="tray_joint" type="fixed">
-    <parent link="${tf_prefix}base_link" />
-    <child link="${tf_prefix}tray_link" />
-    <origin xyz="0 0 ${-(base_radius + tray_height/2)}" rpy="0 0 0" />
-  </joint>
-  <link name="${tf_prefix}tray_link">
-    <xacro:add_box color="White" xyz="0 0 0" rpy="0 0 0" x="${tray_length}" y="${tray_width}" z="${tray_height}" />
-  </link>
-  <!-- Hull -->
-  <joint name="hull_joint" type="fixed">
-    <parent link="${tf_prefix}base_link" />
-    <child link="${tf_prefix}hull_link" />
-    <origin xyz="${(base_length-2*base_radius)/2} 0 0" rpy="0 0 0" />
-  </joint>
-  <link name="${tf_prefix}hull_link">
-    <xacro:add_sphere color="Blue" xyz="0 0 0" rpy="0 0 0" radius="${base_radius}" />
-  </link>
-  <!-- Thruster -->
-  <joint name="thruster_joint" type="fixed">
-    <parent link="${tf_prefix}base_link" />
-    <child link="${tf_prefix}thruster_link" />
-    <origin xyz="${-(base_length-2*base_radius)/2} 0 0" rpy="0 0 0" />
-  </joint>
-  <link name="${tf_prefix}thruster_link">
-    <xacro:add_cylinder color="Gray" xyz="0 0 0" rpy="0 ${radians(90)} 0"
-      radius="${base_radius*0.9}" length="${2*base_radius}" />
-  </link>
-  <!-- Fins -->
   <xacro:fin prefix="top" rpy="0 0 0" />
   <xacro:fin prefix="left" rpy="${radians(120)} 0 0" />

File: coug_description/urdf/rover.gazebo.xacro (robot description, xacro)
@@ -12,5 +12,5 @@
  limitations under the License.
 -->
-<robot name="rover" xmlns:xacro="http://www.ros.org/wiki/xacro">
+<robot name="rover_gazebo" xmlns:xacro="http://www.ros.org/wiki/xacro">
   <xacro:arg name="agent_ns" default="rover1gz" />
   <xacro:property name="agent_ns" value="$(arg agent_ns)" />

File: coug_description/urdf/rover.urdf.xacro (robot description, xacro)
@@ -81,4 +81,10 @@
     </inertial>
   </xacro:macro>
+  <!-- TODO: Compare this with the new 2026 URDF -->
+  <!-- Chassis -->
+  <link name="${tf_prefix}base_link">
+    <xacro:add_box color="LightGray" mass="${base_mass}" xyz="0 0 0" rpy="0 0 0" x="${base_length}" y="${base_width}" z="${base_height}" />
+  </link>
+  <!-- Wheels -->
   <xacro:macro name="wheel" params="prefix xoff y_reflect">
     <joint name="${prefix}_wheel_joint" type="continuous">
@@ -94,10 +100,4 @@
     </link>
   </xacro:macro>
-  <!-- TODO: Compare this with the new 2026 URDF -->
-  <!-- Chassis -->
-  <link name="${tf_prefix}base_link">
-    <xacro:add_box color="LightGray" mass="${base_mass}" xyz="0 0 0" rpy="0 0 0" x="${base_length}" y="${base_width}" z="${base_height}" />
-  </link>
-  <!-- Wheels -->
   <xacro:wheel prefix="front_left" xoff="${wheel_xoff}" y_reflect="1" />
   <xacro:wheel prefix="front_right" xoff="${wheel_xoff}" y_reflect="-1" />

File: coug_description/urdf/wamv.gazebo.xacro (robot description, xacro)
@@ -12,5 +12,5 @@
  limitations under the License.
 -->
-<robot name="wamv" xmlns:xacro="http://www.ros.org/wiki/xacro">
+<robot name="wamv_gazebo" xmlns:xacro="http://www.ros.org/wiki/xacro">
   <xacro:arg name="agent_ns" default="wamv1gz" />
   <xacro:property name="agent_ns" value="$(arg agent_ns)" />

File: coug_description/urdf/wamv_holoocean.urdf.xacro (robot description, xacro)
@@ -12,5 +12,5 @@
  limitations under the License.
 -->
-<robot name="wamv" xmlns:xacro="http://www.ros.org/wiki/xacro">
+<robot name="wamv_holoocean" xmlns:xacro="http://www.ros.org/wiki/xacro">
   <xacro:arg name="tf_prefix" default="" />
   <xacro:property name="tf_prefix" value="$(arg tf_prefix)" />
