Commit message: Fix for WAM-V URDF

File: coug_description/urdf/wamv_holoocean.urdf.xacro (robot description, xacro)
@@ -84,5 +84,5 @@
     <parent link="base_link"/>
     <child link="truth_link"/>
-    <origin xyz="-0.55 0 0" rpy="0 0 0"/>
+    <origin xyz="0 0 0" rpy="0 0 0"/>
   </joint>
   <link name="truth_link"/>
