Commit message: Add depth cam to couguv holoocean

File: coug_description/urdf/couguv_holoocean.urdf.xacro (robot description, xacro)
@@ -188,3 +188,10 @@
   </joint>
   <link name="camera_link" />
+  <!-- Configured depth camera pose (optical frame) -->
+  <joint name="depth_camera_joint" type="fixed">
+    <parent link="dvl_link" />
+    <child link="depth_camera_link" />
+    <origin xyz="0 0 0" rpy="${pi} 0 ${-pi/2}" />
+  </joint>
+  <link name="depth_camera_link" />
 </robot>
