Commit message: Add sonar link to BlueROV2

File: coug_description/urdf/bluerov2.urdf.xacro (robot description, xacro)
@@ -18,5 +18,5 @@
     </visual>
   </link>
-  <!-- TODO: Add sonar from Braden's URDF, move COM to realistic location -->
+  <!-- TODO: Move COM to realistic location -->
   <!-- IMU Link -->
   <link name="imu_link"/>
@@ -47,3 +47,10 @@
     <origin xyz="-0.27161 -0.10886 -0.01984" rpy="${pi} 0 0"/>
   </joint>
+  <!-- Sonar Link -->
+  <link name="sonar_link"/>
+  <joint name="sonar_joint" type="fixed">
+    <parent link="base_link"/>
+    <child link="sonar_link"/>
+    <origin xyz="0.2 0 0" rpy="0 0 0"/>
+  </joint>
 </robot>

Commit message: WIP WAM-V scenario

File: coug_description/urdf/bluerov2.urdf.xacro (robot description, xacro)
@@ -14,8 +14,31 @@
     <visual>
       <geometry>
-        <mesh filename="package://coug_description/urdf/meshes/bluerov2.dae" scale="0.025 0.025 0.025"/>
+        <mesh filename="package://coug_description/urdf/meshes/bluerov2/bluerov2.dae" scale="0.025 0.025 0.025"/>
       </geometry>
     </visual>
   </link>
+  <xacro:macro name="thruster" params="name xyz rpy mesh vis_rpy">
+    <joint name="${name}_joint" type="fixed">
+      <parent link="base_link"/>
+      <child link="${name}_link"/>
+      <origin xyz="${xyz}" rpy="${rpy}"/>
+    </joint>
+    <link name="${name}_link">
+      <visual>
+        <origin xyz="0 0 0" rpy="${vis_rpy}"/>
+        <geometry>
+          <mesh filename="package://coug_description/urdf/meshes/bluerov2/${mesh}"/>
+        </geometry>
+      </visual>
+    </link>
+  </xacro:macro>
+  <xacro:thruster name="thruster1" xyz="0.14 -0.092 0.0"   rpy="-1.571 1.571 -0.785" mesh="t200_ccw_prop.dae" vis_rpy="-1.571 0 0"/>
+  <xacro:thruster name="thruster2" xyz="0.14 0.092 0.0"    rpy="-1.571 1.571 -2.356" mesh="t200_ccw_prop.dae" vis_rpy="-1.571 0 0"/>
+  <xacro:thruster name="thruster3" xyz="-0.14 -0.092 0.0"  rpy="-1.571 1.571 0.785"  mesh="t200_cw_prop.dae"  vis_rpy="1.571 0 0"/>
+  <xacro:thruster name="thruster4" xyz="-0.14 0.092 0.0"   rpy="-1.571 1.571 2.356"  mesh="t200_cw_prop.dae"  vis_rpy="1.571 0 0"/>
+  <xacro:thruster name="thruster5" xyz="0.118 -0.215 0.064"  rpy="0 0 0" mesh="t200_ccw_prop.dae" vis_rpy="-1.571 0 1.571"/>
+  <xacro:thruster name="thruster6" xyz="0.118 0.215 0.064"   rpy="0 0 0" mesh="t200_cw_prop.dae"  vis_rpy="1.571 0 1.571"/>
+  <xacro:thruster name="thruster7" xyz="-0.118 -0.215 0.064" rpy="0 0 0" mesh="t200_cw_prop.dae"  vis_rpy="1.571 0 1.571"/>
+  <xacro:thruster name="thruster8" xyz="-0.118 0.215 0.064"  rpy="0 0 0" mesh="t200_ccw_prop.dae" vis_rpy="-1.571 0 1.571"/>
   <!-- TODO: Move COM to realistic location -->
   <!-- IMU Link -->

File: coug_description/urdf/bluerov2_holoocean.urdf.xacro (robot description, xacro)
@@ -15,8 +15,31 @@
     <visual>
       <geometry>
-        <mesh filename="package://coug_description/urdf/meshes/bluerov2.dae" scale="0.025 0.025 0.025"/>
+        <mesh filename="package://coug_description/urdf/meshes/bluerov2/bluerov2.dae" scale="0.025 0.025 0.025"/>
       </geometry>
     </visual>
   </link>
+  <xacro:macro name="thruster" params="name xyz rpy mesh vis_rpy">
+    <joint name="${name}_joint" type="fixed">
+      <parent link="base_link"/>
+      <child link="${name}_link"/>
+      <origin xyz="${xyz}" rpy="${rpy}"/>
+    </joint>
+    <link name="${name}_link">
+      <visual>
+        <origin xyz="0 0 0" rpy="${vis_rpy}"/>
+        <geometry>
+          <mesh filename="package://coug_description/urdf/meshes/bluerov2/${mesh}"/>
+        </geometry>
+      </visual>
+    </link>
+  </xacro:macro>
+  <xacro:thruster name="thruster1" xyz="0.14 -0.092 0.0"   rpy="-1.571 1.571 -0.785" mesh="t200_ccw_prop.dae" vis_rpy="-1.571 0 0"/>
+  <xacro:thruster name="thruster2" xyz="0.14 0.092 0.0"    rpy="-1.571 1.571 -2.356" mesh="t200_ccw_prop.dae" vis_rpy="-1.571 0 0"/>
+  <xacro:thruster name="thruster3" xyz="-0.14 -0.092 0.0"  rpy="-1.571 1.571 0.785"  mesh="t200_cw_prop.dae"  vis_rpy="1.571 0 0"/>
+  <xacro:thruster name="thruster4" xyz="-0.14 0.092 0.0"   rpy="-1.571 1.571 2.356"  mesh="t200_cw_prop.dae"  vis_rpy="1.571 0 0"/>
+  <xacro:thruster name="thruster5" xyz="0.118 -0.215 0.064"  rpy="0 0 0" mesh="t200_ccw_prop.dae" vis_rpy="-1.571 0 1.571"/>
+  <xacro:thruster name="thruster6" xyz="0.118 0.215 0.064"   rpy="0 0 0" mesh="t200_cw_prop.dae"  vis_rpy="1.571 0 1.571"/>
+  <xacro:thruster name="thruster7" xyz="-0.118 -0.215 0.064" rpy="0 0 0" mesh="t200_cw_prop.dae"  vis_rpy="1.571 0 1.571"/>
+  <xacro:thruster name="thruster8" xyz="-0.118 0.215 0.064"  rpy="0 0 0" mesh="t200_ccw_prop.dae" vis_rpy="-1.571 0 1.571"/>
   <!-- NOTE: These are exact HoloOcean socket locations as of 2.0.1 -->
   <!-- COM -->

File: coug_description/urdf/turtlmap.urdf.xacro (robot description, xacro)
@@ -14,8 +14,31 @@
     <visual>
       <geometry>
-        <mesh filename="package://coug_description/urdf/meshes/bluerov2.dae" scale="0.025 0.025 0.025"/>
+        <mesh filename="package://coug_description/urdf/meshes/bluerov2/bluerov2.dae" scale="0.025 0.025 0.025"/>
       </geometry>
     </visual>
   </link>
+  <xacro:macro name="thruster" params="name xyz rpy mesh vis_rpy">
+    <joint name="${name}_joint" type="fixed">
+      <parent link="base_link"/>
+      <child link="${name}_link"/>
+      <origin xyz="${xyz}" rpy="${rpy}"/>
+    </joint>
+    <link name="${name}_link">
+      <visual>
+        <origin xyz="0 0 0" rpy="${vis_rpy}"/>
+        <geometry>
+          <mesh filename="package://coug_description/urdf/meshes/bluerov2/${mesh}"/>
+        </geometry>
+      </visual>
+    </link>
+  </xacro:macro>
+  <xacro:thruster name="thruster1" xyz="0.14 -0.092 0.0"   rpy="-1.571 1.571 -0.785" mesh="t200_ccw_prop.dae" vis_rpy="-1.571 0 0"/>
+  <xacro:thruster name="thruster2" xyz="0.14 0.092 0.0"    rpy="-1.571 1.571 -2.356" mesh="t200_ccw_prop.dae" vis_rpy="-1.571 0 0"/>
+  <xacro:thruster name="thruster3" xyz="-0.14 -0.092 0.0"  rpy="-1.571 1.571 0.785"  mesh="t200_cw_prop.dae"  vis_rpy="1.571 0 0"/>
+  <xacro:thruster name="thruster4" xyz="-0.14 0.092 0.0"   rpy="-1.571 1.571 2.356"  mesh="t200_cw_prop.dae"  vis_rpy="1.571 0 0"/>
+  <xacro:thruster name="thruster5" xyz="0.118 -0.215 0.064"  rpy="0 0 0" mesh="t200_ccw_prop.dae" vis_rpy="-1.571 0 1.571"/>
+  <xacro:thruster name="thruster6" xyz="0.118 0.215 0.064"   rpy="0 0 0" mesh="t200_cw_prop.dae"  vis_rpy="1.571 0 1.571"/>
+  <xacro:thruster name="thruster7" xyz="-0.118 -0.215 0.064" rpy="0 0 0" mesh="t200_cw_prop.dae"  vis_rpy="1.571 0 1.571"/>
+  <xacro:thruster name="thruster8" xyz="-0.118 0.215 0.064"  rpy="0 0 0" mesh="t200_ccw_prop.dae" vis_rpy="-1.571 0 1.571"/>
   <!-- IMU Link -->
   <link name="imu_link"/>

Commit message: Better WAM-V socket designations

File: coug_description/urdf/bluerov2.urdf.xacro (robot description, xacro)
@@ -41,5 +41,4 @@
   <xacro:thruster name="thruster7" xyz="-0.118 -0.215 0.064" rpy="0 0 0" mesh="t200_cw_prop.dae"  vis_rpy="1.571 0 1.571"/>
   <xacro:thruster name="thruster8" xyz="-0.118 0.215 0.064"  rpy="0 0 0" mesh="t200_ccw_prop.dae" vis_rpy="-1.571 0 1.571"/>
-  <!-- TODO: Move COM to realistic location -->
   <!-- IMU Link -->
   <link name="imu_link"/>

File: coug_description/urdf/wamv_holoocean.urdf.xacro (robot description, xacro)
@@ -67,11 +67,11 @@
   </joint>
   <link name="imu_link"/>
-  <joint name="depth_joint" type="fixed">
+  <!-- Payload -->
+   <joint name="depth_joint" type="fixed">
     <parent link="com_link"/>
     <child link="depth_link"/>
-    <origin xyz="0 0 0" rpy="0 0 0"/>
+    <origin xyz="0 0 0" rpy="0 ${pi/2} 0"/>
   </joint>
   <link name="depth_link"/>
-  <!-- Payload -->
   <joint name="dvl_joint" type="fixed">
     <parent link="com_link"/>

Commit message: Fix for DVL FRD frame

File: coug_description/urdf/bluerov2.urdf.xacro (robot description, xacro)
@@ -76,5 +76,6 @@
     <parent link="base_link" />
     <child link="dvl_link" />
-    <origin xyz="-0.27161 -0.10886 -0.01984" rpy="${pi} 0 0" />
+    <!-- Sensor FLU frame; FRD data converted by dvl_a50_twist/dvl_a50_odom -->
+    <origin xyz="-0.27161 -0.10886 -0.01984" rpy="0 0 0" />
   </joint>
   <!-- Sonar Link -->

File: coug_description/urdf/bluerov2_holoocean.urdf.xacro (robot description, xacro)
@@ -68,5 +68,5 @@
     <parent link="com_link" />
     <child link="modem_link" />
-    <!-- FLU frame defined here; seatrac_x150_imu_depth/base_status_poller convert FRD data -->
+    <!-- Sensor FLU frame; FRD data converted by seatrac_x150_imu_depth/base_status_poller -->
     <origin xyz="0 0 0" rpy="0 0 0" />
   </joint>
@@ -91,4 +91,5 @@
     <parent link="com_link" />
     <child link="dvl_link" />
+    <!-- Sensor FLU frame; FRD data converted by dvl_a50_twist/dvl_a50_odom -->
     <origin xyz="0 -0.1 -0.1" rpy="0 0 0" />
   </joint>

File: coug_description/urdf/couguv.urdf.xacro (robot description, xacro)
@@ -149,5 +149,5 @@
     <parent link="base_link" />
     <child link="modem_link" />
-    <!-- FLU frame defined here; seatrac_x150_imu_depth/base_status_poller convert FRD data -->
+    <!-- Sensor FLU frame; FRD data converted by seatrac_x150_imu_depth/base_status_poller -->
     <origin xyz="0.35 0 -0.086" rpy="0 0 0" />
   </joint>
@@ -157,5 +157,6 @@
     <parent link="base_link" />
     <child link="dvl_link" />
-    <origin xyz="0.475 0 -0.035" rpy="${pi} 0 0" />
+    <!-- Sensor FLU frame; FRD data converted by dvl_a50_twist/dvl_a50_odom -->
+    <origin xyz="0.475 0 -0.035" rpy="0 0 0" />
   </joint>
   <link name="dvl_link" />

File: coug_description/urdf/couguv_holoocean.urdf.xacro (robot description, xacro)
@@ -162,5 +162,5 @@
     <parent link="com_link" />
     <child link="modem_link" />
-    <!-- FLU frame defined here; seatrac_x150_imu_depth/base_status_poller convert FRD data -->
+    <!-- Sensor FLU frame; FRD data converted by seatrac_x150_imu_depth/base_status_poller -->
     <origin xyz="0.3785 0 -0.0985" rpy="0 0 0" />
   </joint>
@@ -170,4 +170,5 @@
     <parent link="com_link" />
     <child link="dvl_link" />
+    <!-- Sensor FLU frame; FRD data converted by dvl_a50_twist/dvl_a50_odom -->
     <origin xyz="0.504 0 -0.053" rpy="0 0 0" />
   </joint>

File: coug_description/urdf/turtlmap.urdf.xacro (robot description, xacro)
@@ -55,4 +55,5 @@
     <parent link="base_link" />
     <child link="imu_link" />
+    <!-- Sensor FRD frame -->
     <origin xyz="0 0 0" rpy="${pi/2} 0 ${pi/2}" />
   </joint>
@@ -69,5 +70,6 @@
     <parent link="base_link" />
     <child link="dvl_link" />
-    <origin xyz="0.113 0.001 -0.04" rpy="${pi} 0 0" />
+    <!-- Sensor FLU frame; FRD data converted by dvl_a50_twist/dvl_a50_odom -->
+    <origin xyz="0.113 0.001 -0.04" rpy="0 0 0" />
   </joint>
 </robot>

File: coug_description/urdf/wamv_holoocean.urdf.xacro (robot description, xacro)
@@ -58,4 +58,5 @@
     <parent link="base_link" />
     <child link="dvl_link" />
+    <!-- Sensor FLU frame; FRD data converted by dvl_a50_twist/dvl_a50_odom -->
     <origin xyz="0 0 0" rpy="0 ${pi/2} 0" />
   </joint>
@@ -64,5 +65,5 @@
     <parent link="base_link" />
     <child link="modem_link" />
-    <!-- FLU frame defined here; seatrac_x150_imu_depth/base_status_poller convert FRD data -->
+    <!-- Sensor FLU frame; FRD data converted by seatrac_x150_imu_depth/base_status_poller -->
     <origin xyz="0 0 0" rpy="0 ${pi/2} 0" />
   </joint>

Commit message: Added DVL beam URDF links

File: coug_description/urdf/bluerov2.urdf.xacro (robot description, xacro)
@@ -76,7 +76,20 @@
     <parent link="base_link" />
     <child link="dvl_link" />
-    <!-- Sensor FLU frame; FRD data converted by dvl_a50_twist/dvl_a50_odom -->
+    <!-- Sensor FLU frame; FRD data converted by dvl_a50_twist_beams/dvl_a50_odom -->
     <origin xyz="-0.27161 -0.10886 -0.01984" rpy="0 0 0" />
   </joint>
+  <xacro:macro name="dvl_beam" params="name yaw">
+    <joint name="${name}_joint" type="fixed">
+      <parent link="dvl_link" />
+      <child link="${name}_link" />
+      <!-- +X axis down each DVL beam -->
+      <origin xyz="0 0 0" rpy="0 ${radians(67.5)} ${yaw}" />
+    </joint>
+    <link name="${name}_link" />
+  </xacro:macro>
+  <xacro:dvl_beam name="beam0" yaw="${radians(-135)}" />
+  <xacro:dvl_beam name="beam1" yaw="${radians(135)}" />
+  <xacro:dvl_beam name="beam2" yaw="${radians(45)}" />
+  <xacro:dvl_beam name="beam3" yaw="${radians(-45)}" />
   <!-- Sonar Link -->
   <link name="sonar_link" />

File: coug_description/urdf/bluerov2_holoocean.urdf.xacro (robot description, xacro)
@@ -91,8 +91,21 @@
     <parent link="com_link" />
     <child link="dvl_link" />
-    <!-- Sensor FLU frame; FRD data converted by dvl_a50_twist/dvl_a50_odom -->
+    <!-- Sensor FLU frame; FRD data converted by dvl_a50_twist_beams/dvl_a50_odom -->
     <origin xyz="0 -0.1 -0.1" rpy="0 0 0" />
   </joint>
   <link name="dvl_link" />
+  <xacro:macro name="dvl_beam" params="name yaw">
+    <joint name="${name}_joint" type="fixed">
+      <parent link="dvl_link" />
+      <child link="${name}_link" />
+      <!-- +X axis down each DVL beam -->
+      <origin xyz="0 0 0" rpy="0 ${radians(67.5)} ${yaw}" />
+    </joint>
+    <link name="${name}_link" />
+  </xacro:macro>
+  <xacro:dvl_beam name="beam0" yaw="${radians(0)}" />
+  <xacro:dvl_beam name="beam1" yaw="${radians(90)}" />
+  <xacro:dvl_beam name="beam2" yaw="${radians(180)}" />
+  <xacro:dvl_beam name="beam3" yaw="${radians(-90)}" />
   <!-- CameraSocket -->
   <joint name="camera_joint" type="fixed">

File: coug_description/urdf/couguv.urdf.xacro (robot description, xacro)
@@ -157,7 +157,20 @@
     <parent link="base_link" />
     <child link="dvl_link" />
-    <!-- Sensor FLU frame; FRD data converted by dvl_a50_twist/dvl_a50_odom -->
+    <!-- Sensor FLU frame; FRD data converted by dvl_a50_twist_beams/dvl_a50_odom -->
     <origin xyz="0.475 0 -0.035" rpy="0 0 0" />
   </joint>
   <link name="dvl_link" />
+  <xacro:macro name="dvl_beam" params="name yaw">
+    <joint name="${name}_joint" type="fixed">
+      <parent link="dvl_link" />
+      <child link="${name}_link" />
+      <!-- +X axis down each DVL beam -->
+      <origin xyz="0 0 0" rpy="0 ${radians(67.5)} ${yaw}" />
+    </joint>
+    <link name="${name}_link" />
+  </xacro:macro>
+  <xacro:dvl_beam name="beam0" yaw="${radians(-135)}" />
+  <xacro:dvl_beam name="beam1" yaw="${radians(135)}" />
+  <xacro:dvl_beam name="beam2" yaw="${radians(45)}" />
+  <xacro:dvl_beam name="beam3" yaw="${radians(-45)}" />
 </robot>

File: coug_description/urdf/couguv_holoocean.urdf.xacro (robot description, xacro)
@@ -170,8 +170,21 @@
     <parent link="com_link" />
     <child link="dvl_link" />
-    <!-- Sensor FLU frame; FRD data converted by dvl_a50_twist/dvl_a50_odom -->
+    <!-- Sensor FLU frame; FRD data converted by dvl_a50_twist_beams/dvl_a50_odom -->
     <origin xyz="0.504 0 -0.053" rpy="0 0 0" />
   </joint>
   <link name="dvl_link" />
+  <xacro:macro name="dvl_beam" params="name yaw">
+    <joint name="${name}_joint" type="fixed">
+      <parent link="dvl_link" />
+      <child link="${name}_link" />
+      <!-- +X axis down each DVL beam -->
+      <origin xyz="0 0 0" rpy="0 ${radians(67.5)} ${yaw}" />
+    </joint>
+    <link name="${name}_link" />
+  </xacro:macro>
+  <xacro:dvl_beam name="beam0" yaw="${radians(0)}" />
+  <xacro:dvl_beam name="beam1" yaw="${radians(90)}" />
+  <xacro:dvl_beam name="beam2" yaw="${radians(180)}" />
+  <xacro:dvl_beam name="beam3" yaw="${radians(-90)}" />
   <!-- CameraSocket -->
   <joint name="camera_joint" type="fixed">

File: coug_description/urdf/turtlmap.urdf.xacro (robot description, xacro)
@@ -70,6 +70,19 @@
     <parent link="base_link" />
     <child link="dvl_link" />
-    <!-- Sensor FLU frame; FRD data converted by dvl_a50_twist/dvl_a50_odom -->
+    <!-- Sensor FLU frame; FRD data converted by dvl_a50_twist_beams/dvl_a50_odom -->
     <origin xyz="0.113 0.001 -0.04" rpy="0 0 0" />
   </joint>
+  <xacro:macro name="dvl_beam" params="name yaw">
+    <joint name="${name}_joint" type="fixed">
+      <parent link="dvl_link" />
+      <child link="${name}_link" />
+      <!-- +X axis down each DVL beam -->
+      <origin xyz="0 0 0" rpy="0 ${radians(67.5)} ${yaw}" />
+    </joint>
+    <link name="${name}_link" />
+  </xacro:macro>
+  <xacro:dvl_beam name="beam0" yaw="${radians(-135)}" />
+  <xacro:dvl_beam name="beam1" yaw="${radians(135)}" />
+  <xacro:dvl_beam name="beam2" yaw="${radians(45)}" />
+  <xacro:dvl_beam name="beam3" yaw="${radians(-45)}" />
 </robot>

File: coug_description/urdf/wamv_holoocean.urdf.xacro (robot description, xacro)
@@ -58,8 +58,21 @@
     <parent link="base_link" />
     <child link="dvl_link" />
-    <!-- Sensor FLU frame; FRD data converted by dvl_a50_twist/dvl_a50_odom -->
-    <origin xyz="0 0 0" rpy="0 ${pi/2} 0" />
+    <!-- Sensor FLU frame; FRD data converted by dvl_a50_twist_beams/dvl_a50_odom -->
+    <origin xyz="0 0 0" rpy="0 0 0" />
   </joint>
   <link name="dvl_link" />
+  <xacro:macro name="dvl_beam" params="name yaw">
+    <joint name="${name}_joint" type="fixed">
+      <parent link="dvl_link" />
+      <child link="${name}_link" />
+      <!-- +X axis down each DVL beam -->
+      <origin xyz="0 0 0" rpy="0 ${radians(67.5)} ${yaw}" />
+    </joint>
+    <link name="${name}_link" />
+  </xacro:macro>
+  <xacro:dvl_beam name="beam0" yaw="${radians(0)}" />
+  <xacro:dvl_beam name="beam1" yaw="${radians(90)}" />
+  <xacro:dvl_beam name="beam2" yaw="${radians(180)}" />
+  <xacro:dvl_beam name="beam3" yaw="${radians(-90)}" />
   <joint name="modem_joint" type="fixed">
     <parent link="base_link" />

Commit message: Add ZED frame

File: coug_description/urdf/bluerov2.urdf.xacro (robot description, xacro)
@@ -45,5 +45,4 @@
     vis_rpy="-1.571 0 1.571" />
   <!-- IMU Link -->
-  <link name="imu_link" />
   <joint name="imu_joint" type="fixed">
     <parent link="base_link" />
@@ -51,6 +50,6 @@
     <origin xyz="0 0 0" rpy="0 0 0" />
   </joint>
+  <link name="imu_link" />
   <!-- Depth Link -->
-  <link name="depth_link" />
   <joint name="depth_joint" type="fixed">
     <parent link="base_link" />
@@ -58,6 +57,6 @@
     <origin xyz="0 0 0" rpy="0 0 0" />
   </joint>
+  <link name="depth_link" />
   <!-- GPS Link -->
-  <link name="gps_link" />
   <joint name="gps_joint" type="fixed">
     <parent link="base_link" />
@@ -65,6 +64,6 @@
     <origin xyz="-0.11770 -0.20723 0.40019" rpy="0 0 0" />
   </joint>
+  <link name="gps_link" />
   <!-- DVL Link -->
-  <link name="dvl_link" />
   <joint name="dvl_joint" type="fixed">
     <parent link="base_link" />
@@ -73,4 +72,5 @@
     <origin xyz="-0.27161 -0.10886 -0.01984" rpy="0 0 0" />
   </joint>
+  <link name="dvl_link" />
   <xacro:macro name="dvl_beam" params="name yaw">
     <joint name="${name}_joint" type="fixed">
@@ -87,5 +87,4 @@
   <xacro:dvl_beam name="beam3" yaw="${radians(-45)}" />
   <!-- Sonar Link -->
-  <link name="sonar_link" />
   <joint name="sonar_joint" type="fixed">
     <parent link="base_link" />
@@ -93,3 +92,4 @@
     <origin xyz="0.2 0 0" rpy="0 0 0" />
   </joint>
+  <link name="sonar_link" />
 </robot>

File: coug_description/urdf/bluerov2_holoocean.urdf.xacro (robot description, xacro)
@@ -116,7 +116,5 @@
   </joint>
   <link name="sonar_link" />
-  <!-- Configured stereo camera poses -->
-  <!-- In HoloOcean, cameras look along X, with Z up and Y left -->
-  <!-- In ROS 2, cameras look along Z, with X right and Y down -->
+  <!-- Configured stereo camera poses (optical frame) -->
   <joint name="front_stereo_joint" type="fixed">
     <parent link="dvl_link" />

File: coug_description/urdf/turtlmap.urdf.xacro (robot description, xacro)
@@ -45,5 +45,4 @@
     vis_rpy="-1.571 0 1.571" />
   <!-- IMU Link -->
-  <link name="imu_link" />
   <joint name="imu_joint" type="fixed">
     <parent link="base_link" />
@@ -52,6 +51,6 @@
     <origin xyz="0 0 0" rpy="${pi/2} 0 ${pi/2}" />
   </joint>
+  <link name="imu_link" />
   <!-- Depth Link -->
-  <link name="depth_link" />
   <joint name="depth_joint" type="fixed">
     <parent link="base_link" />
@@ -59,6 +58,6 @@
     <origin xyz="0 0 0" rpy="0 0 0" />
   </joint>
+  <link name="depth_link" />
   <!-- DVL Link -->
-  <link name="dvl_link" />
   <joint name="dvl_joint" type="fixed">
     <parent link="base_link" />
@@ -67,4 +66,5 @@
     <origin xyz="0.113 0.001 -0.04" rpy="0 0 0" />
   </joint>
+  <link name="dvl_link" />
   <xacro:macro name="dvl_beam" params="name yaw">
     <joint name="${name}_joint" type="fixed">
@@ -80,3 +80,10 @@
   <xacro:dvl_beam name="beam2" yaw="${radians(45)}" />
   <xacro:dvl_beam name="beam3" yaw="${radians(-45)}" />
+  <!-- ZED Mini Camera Link -->
+  <joint name="zedm_left_camera_joint" type="fixed">
+    <parent link="imu_link" />
+    <child link="zedm_left_camera_frame" />
+    <origin xyz="0 0 0" rpy="0 0 0" />
+  </joint>
+  <link name="zedm_left_camera_frame" />
 </robot>

Commit message: Change 3D sonar mount to upside down

File: coug_description/urdf/bluerov2.urdf.xacro (robot description, xacro)
@@ -90,5 +90,5 @@
     <parent link="base_link" />
     <child link="sonar_link" />
-    <origin xyz="0.2 0 0" rpy="0 0 0" />
+    <origin xyz="0.2 0 0" rpy="${radians(180)} 0 0" />
   </joint>
   <link name="sonar_link" />

Commit message: Fix for sonar FRD frame

File: coug_description/urdf/bluerov2.urdf.xacro (robot description, xacro)
@@ -90,5 +90,5 @@
     <parent link="base_link" />
     <child link="sonar_link" />
-    <origin xyz="0.2 0 0" rpy="${radians(180)} 0 0" />
+    <origin xyz="0.2 0 0" rpy="0 0 0" />
   </joint>
   <link name="sonar_link" />
