Commit message: Added modem socket to bluerov2

File: coug_description/urdf/bluerov2.urdf.xacro (robot description, xacro)
@@ -51,4 +51,11 @@
   </joint>
   <link name="imu_link" />
+  <!-- GPS Link -->
+  <joint name="gps_joint" type="fixed">
+    <parent link="base_link" />
+    <child link="gps_link" />
+    <origin xyz="-0.11770 -0.20723 0.40019" rpy="0 0 0" />
+  </joint>
+  <link name="gps_link" />
   <!-- Depth Link -->
   <joint name="depth_joint" type="fixed">
@@ -58,11 +65,4 @@
   </joint>
   <link name="depth_link" />
-  <!-- GPS Link -->
-  <joint name="gps_joint" type="fixed">
-    <parent link="base_link" />
-    <child link="gps_link" />
-    <origin xyz="-0.11770 -0.20723 0.40019" rpy="0 0 0" />
-  </joint>
-  <link name="gps_link" />
   <!-- DVL Link -->
   <joint name="dvl_joint" type="fixed">
@@ -86,4 +86,13 @@
   <xacro:dvl_beam name="beam2" yaw="${radians(45)}" />
   <xacro:dvl_beam name="beam3" yaw="${radians(-45)}" />
+  <!-- TODO: Update this -->
+  <!-- Modem Link -->
+  <joint name="modem_joint" type="fixed">
+    <parent link="base_link" />
+    <child link="modem_link" />
+    <!-- Sensor FLU frame; FRD data converted by seatrac_x150_imu_depth/base_status_poller -->
+    <origin xyz="0 0 0" rpy="0 0 0" />
+  </joint>
+  <link name="modem_link" />
   <!-- Sonar Link -->
   <joint name="sonar_joint" type="fixed">

File: coug_description/urdf/couguv.urdf.xacro (robot description, xacro)
@@ -139,12 +139,4 @@
   </joint>
   <link name="depth_link" />
-  <!-- Modem Link -->
-  <joint name="modem_joint" type="fixed">
-    <parent link="base_link" />
-    <child link="modem_link" />
-    <!-- Sensor FLU frame; FRD data converted by seatrac_x150_imu_depth/base_status_poller -->
-    <origin xyz="0.35 0 -0.086" rpy="${radians(180)} 0 0" />
-  </joint>
-  <link name="modem_link" />
   <!-- DVL Link -->
   <joint name="dvl_joint" type="fixed">
@@ -168,3 +160,11 @@
   <xacro:dvl_beam name="beam2" yaw="${radians(45)}" />
   <xacro:dvl_beam name="beam3" yaw="${radians(-45)}" />
+  <!-- Modem Link -->
+  <joint name="modem_joint" type="fixed">
+    <parent link="base_link" />
+    <child link="modem_link" />
+    <!-- Sensor FLU frame; FRD data converted by seatrac_x150_imu_depth/base_status_poller -->
+    <origin xyz="0.35 0 -0.086" rpy="${radians(180)} 0 0" />
+  </joint>
+  <link name="modem_link" />
 </robot>

File: coug_description/urdf/couguv_holoocean.urdf.xacro (robot description, xacro)
@@ -152,12 +152,4 @@
   </joint>
   <link name="depth_link" />
-  <!-- AcousticModemSocket -->
-  <joint name="modem_joint" type="fixed">
-    <parent link="com_link" />
-    <child link="modem_link" />
-    <!-- Sensor FLU frame; FRD data converted by seatrac_x150_imu_depth/base_status_poller -->
-    <origin xyz="0.3785 0 -0.0985" rpy="0 0 0" />
-  </joint>
-  <link name="modem_link" />
   <!-- DVLSocket -->
   <joint name="dvl_joint" type="fixed">
@@ -181,4 +173,12 @@
   <xacro:dvl_beam name="beam2" yaw="${radians(180)}" />
   <xacro:dvl_beam name="beam3" yaw="${radians(-90)}" />
+  <!-- AcousticModemSocket -->
+  <joint name="modem_joint" type="fixed">
+    <parent link="com_link" />
+    <child link="modem_link" />
+    <!-- Sensor FLU frame; FRD data converted by seatrac_x150_imu_depth/base_status_poller -->
+    <origin xyz="0.3785 0 -0.0985" rpy="0 0 0" />
+  </joint>
+  <link name="modem_link" />
   <!-- CameraSocket -->
   <joint name="camera_joint" type="fixed">
