Commit message: Better rover URDF noise values

File: coug_description/urdf/bluerov2.urdf.xacro (robot description, xacro)
@@ -65,5 +65,5 @@
     <parent link="base_link" />
     <child link="dvl_link" />
-    <!-- Sensor FLU frame; FRD data converted by dvl_a50_twist_beams/dvl_a50_odom -->
+    <!-- Sensor FLU frame; FRD data converted upstream -->
     <origin xyz="-0.27161 -0.10886 -0.01984" rpy="0 0 0" />
   </joint>
@@ -86,5 +86,5 @@
     <parent link="base_link" />
     <child link="modem_link" />
-    <!-- Sensor FLU frame; FRD data converted by seatrac_x150_imu_depth/base_status_poller -->
+    <!-- Sensor FLU frame; FRD data converted upstream -->
     <origin xyz="0 0 0" rpy="0 0 0" />
   </joint>

File: coug_description/urdf/bluerov2_holoocean.urdf.xacro (robot description, xacro)
@@ -60,5 +60,5 @@
     <parent link="com_link" />
     <child link="modem_link" />
-    <!-- Sensor FLU frame; FRD data converted by seatrac_x150_imu_depth/base_status_poller -->
+    <!-- Sensor FLU frame; FRD data converted upstream -->
     <origin xyz="0 0 0" rpy="0 0 0" />
   </joint>
@@ -83,5 +83,5 @@
     <parent link="com_link" />
     <child link="dvl_link" />
-    <!-- Sensor FLU frame; FRD data converted by dvl_a50_twist_beams/dvl_a50_odom -->
+    <!-- Sensor FLU frame; FRD data converted upstream -->
     <origin xyz="0 -0.1 -0.1" rpy="0 0 0" />
   </joint>

File: coug_description/urdf/couguv.urdf.xacro (robot description, xacro)
@@ -153,5 +153,5 @@
     <parent link="base_link" />
     <child link="dvl_link" />
-    <!-- Sensor FLU frame; FRD data converted by dvl_a50_twist_beams/dvl_a50_odom -->
+    <!-- Sensor FLU frame; FRD data converted upstream -->
     <origin xyz="0.475 0 -0.035" rpy="0 0 0" />
   </joint>
@@ -173,5 +173,5 @@
     <parent link="base_link" />
     <child link="modem_link" />
-    <!-- Sensor FLU frame; FRD data converted by seatrac_x150_imu_depth/base_status_poller -->
+    <!-- Sensor FLU frame; FRD data converted upstream -->
     <origin xyz="0.35 0 -0.086" rpy="${radians(180)} 0 0" />
   </joint>

File: coug_description/urdf/couguv_holoocean.urdf.xacro (robot description, xacro)
@@ -170,5 +170,5 @@
     <parent link="com_link" />
     <child link="dvl_link" />
-    <!-- Sensor FLU frame; FRD data converted by dvl_a50_twist_beams/dvl_a50_odom -->
+    <!-- Sensor FLU frame; FRD data converted upstream -->
     <origin xyz="0.504 0 -0.053" rpy="0 0 0" />
   </joint>
@@ -191,5 +191,5 @@
     <parent link="com_link" />
     <child link="modem_link" />
-    <!-- Sensor FLU frame; FRD data converted by seatrac_x150_imu_depth/base_status_poller -->
+    <!-- Sensor FLU frame; FRD data converted upstream -->
     <origin xyz="0.3785 0 -0.0985" rpy="0 0 0" />
   </joint>

File: coug_description/urdf/rover.urdf.xacro (robot description, xacro)
@@ -66,5 +66,5 @@
     </inertial>
   </xacro:macro>
-  <xacro:macro name="add_imu_noise" params="stddev">
+  <xacro:macro name="add_xyz_noise" params="stddev">
     <xacro:macro name="add_axis_noise">
       <noise type="gaussian">
@@ -161,8 +161,8 @@
     <plugin filename="gz-sim-odometry-publisher-system" name="gz::sim::systems::OdometryPublisher">
       <dimensions>3</dimensions>
-      <!-- https://github.com/stereolabs/zed-ros2-wrapper/blob/v5.4.1/zed_wrapper/config/zed2i.yaml#L11 -->
       <odom_publish_frequency>60</odom_publish_frequency>
       <odom_topic>/${agent_ns}/camera/odom</odom_topic>
       <odom_covariance_topic>/${agent_ns}/camera/odom_with_covariance</odom_covariance_topic>
+      <gaussian_noise>0.01</gaussian_noise>
       <odom_frame>${agent_ns}/odom</odom_frame>
       <robot_base_frame>${agent_ns}/base_link</robot_base_frame>
@@ -174,20 +174,17 @@
       <always_on>true</always_on>
       <update_rate>100</update_rate>
-      <topic>/${agent_ns}/camera/imu/data</topic>
+      <topic>/${agent_ns}/camera/imu/data_raw</topic>
       <gz_frame_id>${agent_ns}/imu_link</gz_frame_id>
       <imu>
-        <enable_orientation>true</enable_orientation>
-        <orientation_reference_frame>
-          <localization>ENU</localization>
-        </orientation_reference_frame>
+        <enable_orientation>false</enable_orientation>
         <!-- 0.007 °/s/√Hz * √100 Hz -> 1.2e-3 rad/s
-          0.0016 m/s^2/√Hz * √100 Hz -> 1.6e-2 m/s^2
-          https://github.com/stereolabs/zed-sdk/issues/487
-          https://github.com/stereolabs/zed-ros2-wrapper/blob/v5.4.1/zed_wrapper/config/common_stereo.yaml#L64 -->
+        0.0016 m/s^2/√Hz * √100 Hz -> 1.6e-2 m/s^2
+        https://github.com/stereolabs/zed-sdk/issues/487
+        https://github.com/stereolabs/zed-ros2-wrapper/blob/v5.4.1/zed_wrapper/config/common_stereo.yaml -->
         <angular_velocity>
-          <xacro:add_imu_noise stddev="1.2e-3" />
+          <xacro:add_xyz_noise stddev="1.2e-3" />
         </angular_velocity>
         <linear_acceleration>
-          <xacro:add_imu_noise stddev="1.6e-2" />
+          <xacro:add_xyz_noise stddev="1.6e-2" />
         </linear_acceleration>
       </imu>
@@ -198,4 +195,8 @@
       <topic>/${agent_ns}/camera/imu/mag</topic>
       <gz_frame_id>${agent_ns}/imu_link</gz_frame_id>
+      <magnetometer>
+        <!-- https://support.sbg-systems.com/sc/el/latest/ellipse-documentation/hardware-documentation/aiding-sensors -->
+        <xacro:add_xyz_noise stddev="3.0e-7" />
+      </magnetometer>
     </sensor>
   </gazebo>
@@ -235,7 +236,7 @@
       <camera>
         <!-- https://www.stereolabs.com/en-us/products/zed-2i
-          https://github.com/stereolabs/zed-ros2-wrapper/blob/v5.4.1/zed_wrapper/config/zed2i.yaml#L10-L20
-          https://github.com/stereolabs/zed-ros2-wrapper/blob/v5.4.1/zed_wrapper/config/common_stereo.yaml#L30-L33
-          https://support.stereolabs.com/articles/9175329825 -->
+        https://github.com/stereolabs/zed-ros2-wrapper/blob/v5.4.1/zed_wrapper/config/zed2i.yaml
+        https://github.com/stereolabs/zed-ros2-wrapper/blob/v5.4.1/zed_wrapper/config/common_stereo.yaml
+        https://support.stereolabs.com/articles/9175329825 -->
         <horizontal_fov>${radians(110)}</horizontal_fov>
         <!-- <horizontal_fov>${radians(68)}</horizontal_fov> -->

File: coug_description/urdf/turtlmap.urdf.xacro (robot description, xacro)
@@ -60,5 +60,5 @@
     <parent link="base_link" />
     <child link="dvl_link" />
-    <!-- Sensor FLU frame; FRD data converted by dvl_a50_twist_beams/dvl_a50_odom -->
+    <!-- Sensor FLU frame; FRD data converted upstream -->
     <origin xyz="0.113 0.001 -0.04" rpy="0 0 0" />
   </joint>

File: coug_description/urdf/wamv_holoocean.urdf.xacro (robot description, xacro)
@@ -51,5 +51,5 @@
     <parent link="base_link" />
     <child link="dvl_link" />
-    <!-- Sensor FLU frame; FRD data converted by dvl_a50_twist_beams/dvl_a50_odom -->
+    <!-- Sensor FLU frame; FRD data converted upstream -->
     <origin xyz="0 0 0" rpy="0 0 0" />
   </joint>
@@ -71,5 +71,5 @@
     <parent link="base_link" />
     <child link="modem_link" />
-    <!-- Sensor FLU frame; FRD data converted by seatrac_x150_imu_depth/base_status_poller -->
+    <!-- Sensor FLU frame; FRD data converted upstream -->
     <origin xyz="0 0 0" rpy="0 ${radians(90)} 0" />
   </joint>
