Commit message: Break out gazebo file

File: coug_description/urdf/rover.urdf.xacro (robot description, xacro)
@@ -1,6 +1,4 @@
 <?xml version="1.0"?>
 <robot name="rover" xmlns:xacro="http://ros.org/wiki/xacro">
-  <xacro:arg name="agent_ns" default="rover1sim" />
-  <xacro:property name="agent_ns" value="$(arg agent_ns)" />
   <xacro:property name="base_height" value="0.15" />
   <xacro:property name="base_width" value="0.5" />
@@ -66,21 +64,4 @@
     </inertial>
   </xacro:macro>
-  <xacro:macro name="add_xyz_noise" params="stddev">
-    <xacro:macro name="add_axis_noise">
-      <noise type="gaussian">
-        <mean>0.0</mean>
-        <stddev>${stddev}</stddev>
-      </noise>
-    </xacro:macro>
-    <x>
-      <xacro:add_axis_noise />
-    </x>
-    <y>
-      <xacro:add_axis_noise />
-    </y>
-    <z>
-      <xacro:add_axis_noise />
-    </z>
-  </xacro:macro>
   <xacro:macro name="wheel" params="prefix xoff y_reflect">
     <joint name="${prefix}_wheel_joint" type="continuous">
@@ -141,124 +122,3 @@
   </joint>
   <link name="gps_link" />
-  <!-- Gazebo plugins -->
-  <gazebo>
-    <plugin filename="gz-sim-diff-drive-system" name="gz::sim::systems::DiffDrive">
-      <left_joint>front_left_wheel_joint</left_joint>
-      <left_joint>middle_left_wheel_joint</left_joint>
-      <left_joint>rear_left_wheel_joint</left_joint>
-      <right_joint>front_right_wheel_joint</right_joint>
-      <right_joint>middle_right_wheel_joint</right_joint>
-      <right_joint>rear_right_wheel_joint</right_joint>
-      <wheel_separation>${2*wheel_yoff}</wheel_separation>
-      <wheel_radius>${wheel_radius}</wheel_radius>
-      <topic>/${agent_ns}/cmd_vel</topic>
-      <odom_topic>/${agent_ns}/wheel/odom</odom_topic>
-      <child_frame_id>${agent_ns}/base_link</child_frame_id>
-    </plugin>
-    <plugin filename="gz-sim-joint-state-publisher-system" name="gz::sim::systems::JointStatePublisher">
-      <topic>/${agent_ns}/joint_states</topic>
-    </plugin>
-    <plugin filename="gz-sim-odometry-publisher-system" name="gz::sim::systems::OdometryPublisher">
-      <dimensions>3</dimensions>
-      <odom_publish_frequency>60</odom_publish_frequency>
-      <odom_topic>/${agent_ns}/camera/odom</odom_topic>
-      <odom_covariance_topic>/${agent_ns}/camera/odom_with_covariance</odom_covariance_topic>
-      <gaussian_noise>0.01</gaussian_noise>
-      <odom_frame>${agent_ns}/odom</odom_frame>
-      <robot_base_frame>${agent_ns}/base_link</robot_base_frame>
-    </plugin>
-  </gazebo>
-  <!-- Gazebo sensors -->
-  <gazebo reference="imu_link">
-    <sensor name="imu" type="imu">
-      <always_on>true</always_on>
-      <update_rate>100</update_rate>
-      <topic>/${agent_ns}/camera/imu/data_raw</topic>
-      <gz_frame_id>${agent_ns}/imu_link</gz_frame_id>
-      <imu>
-        <enable_orientation>false</enable_orientation>
-        <!-- 0.007 °/s/√Hz * √100 Hz -> 1.2e-3 rad/s
-        0.0016 m/s^2/√Hz * √100 Hz -> 1.6e-2 m/s^2
-        https://github.com/stereolabs/zed-sdk/issues/487
-        https://github.com/stereolabs/zed-ros2-wrapper/blob/v5.4.1/zed_wrapper/config/common_stereo.yaml -->
-        <angular_velocity>
-          <xacro:add_xyz_noise stddev="1.2e-3" />
-        </angular_velocity>
-        <linear_acceleration>
-          <xacro:add_xyz_noise stddev="1.6e-2" />
-        </linear_acceleration>
-      </imu>
-    </sensor>
-    <sensor name="magnetometer" type="magnetometer">
-      <always_on>true</always_on>
-      <update_rate>50</update_rate>
-      <topic>/${agent_ns}/camera/imu/mag</topic>
-      <gz_frame_id>${agent_ns}/imu_link</gz_frame_id>
-      <magnetometer>
-        <!-- https://support.sbg-systems.com/sc/el/latest/ellipse-documentation/hardware-documentation/aiding-sensors -->
-        <xacro:add_xyz_noise stddev="3.0e-7" />
-      </magnetometer>
-    </sensor>
-  </gazebo>
-  <gazebo reference="gps_link">
-    <sensor name="gps" type="navsat">
-      <always_on>true</always_on>
-      <update_rate>10</update_rate>
-      <topic>/${agent_ns}/gps/fix</topic>
-      <gz_frame_id>${agent_ns}/gps_link</gz_frame_id>
-      <navsat>
-        <!-- https://content.u-blox.com/sites/default/files/documents/ZED-F9P-01B_DataSheet_UBX-17051259.pdf -->
-        <position_sensing>
-          <horizontal>
-            <noise type="gaussian">
-              <mean>0.0</mean>
-              <!-- Lat/lon degrees, not meters -->
-              <stddev>1.35e-7</stddev>
-            </noise>
-          </horizontal>
-          <vertical>
-            <noise type="gaussian">
-              <mean>0.0</mean>
-              <stddev>0.025</stddev>
-            </noise>
-          </vertical>
-        </position_sensing>
-      </navsat>
-    </sensor>
-  </gazebo>
-  <gazebo reference="depth_camera_link">
-    <sensor name="depth_camera" type="rgbd_camera">
-      <always_on>true</always_on>
-      <!-- <update_rate>60</update_rate> -->
-      <update_rate>20</update_rate>
-      <topic>/${agent_ns}/camera/depth</topic>
-      <gz_frame_id>${agent_ns}/depth_camera_link</gz_frame_id>
-      <camera>
-        <!-- https://www.stereolabs.com/en-us/products/zed-2i
-        https://github.com/stereolabs/zed-ros2-wrapper/blob/v5.4.1/zed_wrapper/config/zed2i.yaml
-        https://github.com/stereolabs/zed-ros2-wrapper/blob/v5.4.1/zed_wrapper/config/common_stereo.yaml
-        https://support.stereolabs.com/articles/9175329825 -->
-        <horizontal_fov>${radians(110)}</horizontal_fov>
-        <!-- <horizontal_fov>${radians(68)}</horizontal_fov> -->
-        <image>
-          <!-- <width>1280</width>
-          <height>720</height> -->
-          <width>640</width>
-          <height>360</height>
-          <format>R8G8B8</format>
-        </image>
-        <clip>
-          <near>0.1</near>
-          <far>100.0</far>
-        </clip>
-        <depth_camera>
-          <clip>
-            <near>0.3</near>
-            <!-- <near>1.5</near> -->
-            <far>15.0</far>
-          </clip>
-        </depth_camera>
-      </camera>
-    </sensor>
-  </gazebo>
 </robot>
