Commit message: Better ZED odom sim

File: coug_description/urdf/rover.gazebo.xacro (robot description, xacro)
@@ -53,6 +53,8 @@
       <odom_covariance_topic>/${agent_ns}/camera/odom_with_covariance</odom_covariance_topic>
       <gaussian_noise>0.01</gaussian_noise>
+      <xyz_offset>${base_length/2 + mast_length/2 + depth_camera_xoff} 0 ${mast_height/2 - base_height/2 + depth_camera_zoff}</xyz_offset>
+      <rpy_offset>0 ${depth_camera_pitch} 0</rpy_offset>
       <odom_frame>${agent_ns}/odom</odom_frame>
-      <robot_base_frame>${agent_ns}/base_link</robot_base_frame>
+      <robot_base_frame>${agent_ns}/depth_camera_link</robot_base_frame>
     </plugin>
   </gazebo>

File: coug_description/urdf/rover.urdf.xacro (robot description, xacro)
@@ -16,4 +16,7 @@
   <xacro:property name="mast_length" value="0.04" />
   <xacro:property name="mast_mass" value="1.5" />
+  <xacro:property name="depth_camera_xoff" value="0.12" />
+  <xacro:property name="depth_camera_zoff" value="0.05" />
+  <xacro:property name="depth_camera_pitch" value="0.1" />
   <material name="LightGray">
     <color rgba="0.8 0.8 0.8 1" />
@@ -101,5 +104,5 @@
     <parent link="mast_link" />
     <child link="depth_camera_link" />
-    <origin xyz="0.12 0 0.05" rpy="0 0.1 0" />
+    <origin xyz="${depth_camera_xoff} 0 ${depth_camera_zoff}" rpy="0 ${depth_camera_pitch} 0" />
   </joint>
   <link name="depth_camera_link" />

Commit message: Start to deal with rover wheel friction

File: coug_description/urdf/rover.gazebo.xacro (robot description, xacro)
@@ -22,4 +22,18 @@
     </z>
   </xacro:macro>
+  <!-- TODO: Add wheel friction that matches the real rover better -->
+  <xacro:macro name="wheel_friction" params="prefix">
+    <gazebo reference="${prefix}_wheel_link">
+      <mu1>1.0</mu1>
+      <mu2>0.5</mu2>
+      <fdir1>1 0 0</fdir1>
+    </gazebo>
+  </xacro:macro>
+  <xacro:wheel_friction prefix="front_left" />
+  <xacro:wheel_friction prefix="front_right" />
+  <xacro:wheel_friction prefix="middle_left" />
+  <xacro:wheel_friction prefix="middle_right" />
+  <xacro:wheel_friction prefix="rear_left" />
+  <xacro:wheel_friction prefix="rear_right" />
   <!-- Gazebo plugins -->
   <gazebo>

Commit message: Add Gazebo WAM-V support

File: coug_description/urdf/rover.gazebo.xacro (robot description, xacro)
@@ -16,22 +16,5 @@
   <xacro:property name="agent_ns" value="$(arg agent_ns)" />
   <xacro:include filename="$(find coug_description)/urdf/rover.urdf.xacro" />
-  <!-- Helpful macros -->
-  <xacro:macro name="add_xyz_noise" params="stddev">
-    <xacro:macro name="add_axis_noise">
-      <noise type="gaussian">
-        <mean>0.0</mean>
-        <stddev>${stddev}</stddev>
-      </noise>
-    </xacro:macro>
-    <x>
-      <xacro:add_axis_noise />
-    </x>
-    <y>
-      <xacro:add_axis_noise />
-    </y>
-    <z>
-      <xacro:add_axis_noise />
-    </z>
-  </xacro:macro>
+  <xacro:include filename="$(find coug_description)/urdf/sensors.gazebo.xacro" />
   <!-- TODO: Add wheel friction that matches the real rover better -->
   <xacro:macro name="wheel_friction" params="prefix">
@@ -66,115 +49,12 @@
       <topic>/${agent_ns}/joint_states</topic>
     </plugin>
-    <plugin filename="gz-sim-odometry-publisher-system" name="gz::sim::systems::OdometryPublisher">
-      <dimensions>3</dimensions>
-      <odom_publish_frequency>60</odom_publish_frequency>
-      <odom_topic>/${agent_ns}/odometry/truth</odom_topic>
-      <odom_frame>map</odom_frame>
-      <robot_base_frame>${agent_ns}/base_link</robot_base_frame>
-    </plugin>
-    <plugin filename="gz-sim-odometry-publisher-system" name="gz::sim::systems::OdometryPublisher">
-      <dimensions>3</dimensions>
-      <odom_publish_frequency>60</odom_publish_frequency>
-      <odom_topic>/${agent_ns}/camera/odom</odom_topic>
-      <odom_covariance_topic>/${agent_ns}/camera/odom_with_covariance</odom_covariance_topic>
-      <gaussian_noise>0.01</gaussian_noise>
-      <xyz_offset>${base_length/2 + mast_length/2 + depth_camera_xoff} 0 ${mast_height/2 - base_height/2 + depth_camera_zoff}</xyz_offset>
-      <rpy_offset>0 ${depth_camera_pitch} 0</rpy_offset>
-      <odom_frame>${agent_ns}/odom</odom_frame>
-      <robot_base_frame>${agent_ns}/depth_camera_link</robot_base_frame>
-    </plugin>
+    <xacro:truth_odometry base_frame="${agent_ns}/base_link" />
+    <xacro:camera_odometry camera_frame="${agent_ns}/depth_camera_link"
+      xyz="${base_length/2 + mast_length/2 + depth_camera_xoff} 0 ${mast_height/2 - base_height/2 + depth_camera_zoff}"
+      rpy="0 ${depth_camera_pitch} 0" />
   </gazebo>
   <!-- Gazebo sensors -->
-  <gazebo reference="imu_link">
-    <sensor name="imu" type="imu">
-      <always_on>true</always_on>
-      <update_rate>100</update_rate>
-      <topic>/${agent_ns}/camera/imu/data_raw</topic>
-      <gz_frame_id>${agent_ns}/imu_link</gz_frame_id>
-      <imu>
-        <enable_orientation>false</enable_orientation>
-        <!-- 0.007 °/s/√Hz * √100 Hz -> 1.2e-3 rad/s
-          0.0016 m/s^2/√Hz * √100 Hz -> 1.6e-2 m/s^2
-          https://github.com/stereolabs/zed-sdk/issues/487
-          https://github.com/stereolabs/zed-ros2-wrapper/blob/v5.4.1/zed_wrapper/config/common_stereo.yaml -->
-        <angular_velocity>
-          <xacro:add_xyz_noise stddev="1.2e-3" />
-        </angular_velocity>
-        <linear_acceleration>
-          <xacro:add_xyz_noise stddev="1.6e-2" />
-        </linear_acceleration>
-      </imu>
-    </sensor>
-    <sensor name="magnetometer" type="magnetometer">
-      <always_on>true</always_on>
-      <update_rate>50</update_rate>
-      <topic>/${agent_ns}/camera/imu/mag</topic>
-      <gz_frame_id>${agent_ns}/imu_link</gz_frame_id>
-      <magnetometer>
-        <!-- https://support.sbg-systems.com/sc/el/latest/ellipse-documentation/hardware-documentation/aiding-sensors -->
-        <xacro:add_xyz_noise stddev="3.0e-7" />
-      </magnetometer>
-    </sensor>
-  </gazebo>
-  <gazebo reference="gps_link">
-    <sensor name="gps" type="navsat">
-      <always_on>true</always_on>
-      <update_rate>10</update_rate>
-      <topic>/${agent_ns}/gps/fix</topic>
-      <gz_frame_id>${agent_ns}/gps_link</gz_frame_id>
-      <navsat>
-        <!-- https://content.u-blox.com/sites/default/files/documents/ZED-F9P-01B_DataSheet_UBX-17051259.pdf -->
-        <position_sensing>
-          <horizontal>
-            <noise type="gaussian">
-              <mean>0.0</mean>
-              <!-- Lat/lon degrees, not meters -->
-              <stddev>1.35e-7</stddev>
-            </noise>
-          </horizontal>
-          <vertical>
-            <noise type="gaussian">
-              <mean>0.0</mean>
-              <stddev>0.025</stddev>
-            </noise>
-          </vertical>
-        </position_sensing>
-      </navsat>
-    </sensor>
-  </gazebo>
-  <gazebo reference="depth_camera_link">
-    <sensor name="depth_camera" type="rgbd_camera">
-      <always_on>true</always_on>
-      <!-- <update_rate>60</update_rate> -->
-      <update_rate>20</update_rate>
-      <topic>/${agent_ns}/camera/depth</topic>
-      <gz_frame_id>${agent_ns}/depth_camera_link</gz_frame_id>
-      <camera>
-        <!-- https://www.stereolabs.com/en-us/products/zed-2i
-          https://github.com/stereolabs/zed-ros2-wrapper/blob/v5.4.1/zed_wrapper/config/zed2i.yaml
-          https://github.com/stereolabs/zed-ros2-wrapper/blob/v5.4.1/zed_wrapper/config/common_stereo.yaml
-          https://support.stereolabs.com/articles/9175329825 -->
-        <horizontal_fov>${radians(110)}</horizontal_fov>
-        <!-- <horizontal_fov>${radians(68)}</horizontal_fov> -->
-        <image>
-          <!-- <width>1280</width>
-            <height>720</height> -->
-          <width>640</width>
-          <height>360</height>
-          <format>R8G8B8</format>
-        </image>
-        <clip>
-          <near>0.1</near>
-          <far>100.0</far>
-        </clip>
-        <depth_camera>
-          <clip>
-            <near>0.3</near>
-            <!-- <near>1.5</near> -->
-            <far>15.0</far>
-          </clip>
-        </depth_camera>
-      </camera>
-    </sensor>
-  </gazebo>
+  <xacro:imu_sensors link="imu_link" frame="${agent_ns}/imu_link" />
+  <xacro:gps_sensor link="gps_link" frame="${agent_ns}/gps_link" />
+  <xacro:depth_camera_sensor link="depth_camera_link" frame="${agent_ns}/depth_camera_link" />
 </robot>

File: coug_description/urdf/wamv_holoocean.urdf.xacro (robot description, xacro)
@@ -13,4 +13,5 @@
 -->
 <robot xmlns:xacro="http://www.ros.org/wiki/xacro" name="wamv">
+  <xacro:include filename="$(find coug_description)/urdf/wamv_platform.xacro" />
   <xacro:property name="mass" value="9.5" />
   <xacro:property name="ixx" value="0.16" />
@@ -20,5 +21,5 @@
     <visual>
       <geometry>
-        <mesh filename="package://coug_description/urdf/meshes/wamv/WAM-V-Base.dae" />
+        <mesh filename="package://wamv_description/models/WAM-V-Base/mesh/WAM-V-Base.dae" />
       </geometry>
     </visual>
@@ -33,5 +34,5 @@
       <visual>
         <geometry>
-          <mesh filename="package://coug_description/urdf/meshes/wamv/engine.dae" />
+          <mesh filename="package://wamv_description/models/engine/mesh/engine.dae" />
         </geometry>
       </visual>
@@ -45,5 +46,5 @@
       <visual>
         <geometry>
-          <mesh filename="package://coug_description/urdf/meshes/wamv/propeller.dae" />
+          <mesh filename="package://wamv_description/models/propeller/mesh/propeller.dae" />
         </geometry>
       </visual>
@@ -88,27 +89,4 @@
   <link name="modem_link" />
   <!-- Platform -->
-  <joint name="gps_joint" type="fixed">
-    <parent link="base_link" />
-    <child link="gps_link" />
-    <origin xyz="0.55 0 1.3" rpy="0 0 0" />
-  </joint>
-  <link name="gps_link" />
-  <joint name="imu_joint" type="fixed">
-    <parent link="base_link" />
-    <child link="imu_link" />
-    <origin xyz="0.55 0 1.3" rpy="0 0 0" />
-  </joint>
-  <link name="imu_link" />
-  <joint name="depth_camera_joint" type="fixed">
-    <parent link="base_link" />
-    <child link="depth_camera_link" />
-    <origin xyz="2.0 0 2.0" rpy="0 ${radians(15)} 0" />
-  </joint>
-  <link name="depth_camera_link" />
-  <joint name="depth_camera_optical_joint" type="fixed">
-    <parent link="depth_camera_link" />
-    <child link="depth_camera_optical_link" />
-    <origin xyz="0 0 0" rpy="${radians(-90)} 0 ${radians(-90)}" />
-  </joint>
-  <link name="depth_camera_optical_link" />
+  <xacro:wamv_platform />
 </robot>
