Commit message: Better WAM-V setup

File: coug_description/urdf/wamv.gazebo.xacro (robot description, xacro)
@@ -15,15 +15,14 @@
   <xacro:arg name="agent_ns" default="wamv1gz" />
   <xacro:property name="agent_ns" value="$(arg agent_ns)" />
-  <xacro:arg name="namespace" default="$(arg agent_ns)" />
-  <xacro:property name="namespace" value="$(arg namespace)" scope="global" />
+  <xacro:arg name="tf_prefix" default="$(arg agent_ns)/" />
+  <xacro:include filename="$(find coug_description)/urdf/wamv.urdf.xacro" />
+  <xacro:include filename="$(find coug_description)/urdf/sensors.gazebo.xacro" />
   <xacro:include filename="$(find wamv_gazebo)/urdf/dynamics/wamv_gazebo_dynamics_plugin.xacro" />
-  <xacro:include filename="$(find wamv_description)/urdf/wamv_base.urdf.xacro" />
-  <xacro:include filename="$(find wamv_gazebo)/urdf/thruster_layouts/wamv_aft_thrusters.xacro" />
   <xacro:usv_dynamics_gazebo name="wamv_dynamics_plugin" />
-  <xacro:include filename="$(find coug_description)/urdf/wamv_platform.xacro" />
-  <xacro:include filename="$(find coug_description)/urdf/sensors.gazebo.xacro" />
-  <xacro:wamv_platform tf_prefix="${namespace}/" />
   <!-- Gazebo plugins -->
   <gazebo>
+    <plugin filename="gz-sim-joint-state-publisher-system" name="gz::sim::systems::JointStatePublisher">
+      <topic>/${agent_ns}/joint_states</topic>
+    </plugin>
     <xacro:truth_odometry base_frame="${agent_ns}/base_link" />
     <xacro:camera_odometry camera_frame="${agent_ns}/depth_camera_link"
@@ -31,6 +30,6 @@
   </gazebo>
   <!-- Gazebo sensors -->
-  <xacro:imu_sensors link="${namespace}/imu_link" frame="${agent_ns}/imu_link" />
-  <xacro:gps_sensor link="${namespace}/gps_link" frame="${agent_ns}/gps_link" />
-  <xacro:depth_camera_sensor link="${namespace}/depth_camera_link" frame="${agent_ns}/depth_camera_link" />
+  <xacro:imu_sensors link="${agent_ns}/imu_link" frame="${agent_ns}/imu_link" />
+  <xacro:gps_sensor link="${agent_ns}/gps_link" frame="${agent_ns}/gps_link" />
+  <xacro:depth_camera_sensor link="${agent_ns}/depth_camera_link" frame="${agent_ns}/depth_camera_link" />
 </robot>

File: coug_description/urdf/wamv_holoocean.urdf.xacro (robot description, xacro)
@@ -15,44 +15,5 @@
   <xacro:arg name="tf_prefix" default="" />
   <xacro:property name="tf_prefix" value="$(arg tf_prefix)" />
-  <xacro:include filename="$(find coug_description)/urdf/wamv_platform.xacro" />
-  <xacro:property name="mass" value="9.5" />
-  <xacro:property name="ixx" value="0.16" />
-  <xacro:property name="iyy" value="0.17" />
-  <xacro:property name="izz" value="0.12" />
-  <link name="${tf_prefix}base_link">
-    <visual>
-      <geometry>
-        <mesh filename="package://wamv_description/models/WAM-V-Base/mesh/WAM-V-Base.dae" />
-      </geometry>
-    </visual>
-  </link>
-  <xacro:macro name="engine" params="prefix y">
-    <joint name="${prefix}_engine_joint" type="fixed">
-      <parent link="${tf_prefix}base_link" />
-      <child link="${tf_prefix}${prefix}_engine_link" />
-      <origin xyz="-2.373776 ${y} 0.318237" rpy="0 0 0" />
-    </joint>
-    <link name="${tf_prefix}${prefix}_engine_link">
-      <visual>
-        <geometry>
-          <mesh filename="package://wamv_description/models/engine/mesh/engine.dae" />
-        </geometry>
-      </visual>
-    </link>
-    <joint name="${prefix}_propeller_joint" type="fixed">
-      <parent link="${tf_prefix}${prefix}_engine_link" />
-      <child link="${tf_prefix}${prefix}_propeller_link" />
-      <origin xyz="-0.278156 0 -0.509371" rpy="0 0 0" />
-    </joint>
-    <link name="${tf_prefix}${prefix}_propeller_link">
-      <visual>
-        <geometry>
-          <mesh filename="package://wamv_description/models/propeller/mesh/propeller.dae" />
-        </geometry>
-      </visual>
-    </link>
-  </xacro:macro>
-  <xacro:engine prefix="left" y="1.027135" />
-  <xacro:engine prefix="right" y="-1.027135" />
+  <xacro:include filename="$(find coug_description)/urdf/wamv.urdf.xacro" />
   <!-- NOTE: These are exact HoloOcean socket locations as of 2.3.0 -->
   <!-- Payload -->
@@ -90,5 +51,3 @@
   </joint>
   <link name="${tf_prefix}modem_link" />
-  <!-- Platform -->
-  <xacro:wamv_platform tf_prefix="${tf_prefix}" />
 </robot>
