Commit message: Better URDFs

File: coug_description/urdf/bluerov2_body.xacro (robot description, xacro)
@@ -13,4 +13,5 @@
 -->
 <robot xmlns:xacro="http://www.ros.org/wiki/xacro">
+  <xacro:include filename="$(find coug_description)/urdf/common.xacro" />
   <link name="${tf_prefix}base_link">
     <visual>
@@ -21,9 +22,5 @@
   </link>
   <xacro:macro name="thruster" params="prefix xyz rpy mesh mesh_rpy">
-    <joint name="${prefix}_joint" type="fixed">
-      <parent link="${tf_prefix}base_link" />
-      <child link="${tf_prefix}${prefix}_link" />
-      <origin xyz="${xyz}" rpy="${rpy}" />
-    </joint>
+    <xacro:fixed_joint name="${prefix}" xyz="${xyz}" rpy="${rpy}" />
     <link name="${tf_prefix}${prefix}_link">
       <visual>

File: coug_description/urdf/common.xacro (robot description, xacro)
@@ -80,5 +80,5 @@
     </xacro:if>
   </xacro:macro>
-  <xacro:macro name="sensor_frame" params="name parent:=base xyz:='0 0 0' rpy:='0 0 0'">
+  <xacro:macro name="fixed_joint" params="name parent:=base xyz:='0 0 0' rpy:='0 0 0'">
     <joint name="${name}_joint" type="fixed">
       <parent link="${tf_prefix}${parent}_link" />
@@ -86,4 +86,7 @@
       <origin xyz="${xyz}" rpy="${rpy}" />
     </joint>
+  </xacro:macro>
+  <xacro:macro name="sensor_frame" params="name parent:=base xyz:='0 0 0' rpy:='0 0 0'">
+    <xacro:fixed_joint name="${name}" parent="${parent}" xyz="${xyz}" rpy="${rpy}" />
     <link name="${tf_prefix}${name}_link" />
   </xacro:macro>

File: coug_description/urdf/couguv_body.xacro (robot description, xacro)
@@ -13,4 +13,5 @@
 -->
 <robot xmlns:xacro="http://www.ros.org/wiki/xacro">
+  <xacro:include filename="$(find coug_description)/urdf/common.xacro" />
   <xacro:property name="base_radius" value="0.06" />
   <xacro:property name="base_length" value="1.2" />
@@ -40,27 +41,15 @@
   <!-- Body -->
   <link name="${tf_prefix}base_link" />
-  <joint name="clear_body_joint" type="fixed">
-    <parent link="${tf_prefix}base_link" />
-    <child link="${tf_prefix}clear_body_link" />
-    <origin xyz="0 0 0" rpy="0 0 0" />
-  </joint>
+  <xacro:fixed_joint name="clear_body" />
   <link name="${tf_prefix}clear_body_link">
     <xacro:cylinder_shape color="Acrylic" radius="${base_radius}" length="${enclosure_length}"
       rpy="0 ${radians(90)} 0" />
   </link>
-  <joint name="front_body_joint" type="fixed">
-    <parent link="${tf_prefix}base_link" />
-    <child link="${tf_prefix}front_body_link" />
-    <origin xyz="${(base_length - 2*base_radius - enclosure_length)/4 + enclosure_length/2} 0 0" rpy="0 0 0" />
-  </joint>
+  <xacro:fixed_joint name="front_body" xyz="${(base_length - 2*base_radius - enclosure_length)/4 + enclosure_length/2} 0 0" />
   <link name="${tf_prefix}front_body_link">
     <xacro:cylinder_shape color="Blue" radius="${base_radius}" length="${(base_length - 2*base_radius - enclosure_length)/2}"
       rpy="0 ${radians(90)} 0" />
   </link>
-  <joint name="back_body_joint" type="fixed">
-    <parent link="${tf_prefix}base_link" />
-    <child link="${tf_prefix}back_body_link" />
-    <origin xyz="${-((base_length - 2*base_radius - enclosure_length)/4 + enclosure_length/2)} 0 0" rpy="0 0 0" />
-  </joint>
+  <xacro:fixed_joint name="back_body" xyz="${-((base_length - 2*base_radius - enclosure_length)/4 + enclosure_length/2)} 0 0" />
   <link name="${tf_prefix}back_body_link">
     <xacro:cylinder_shape color="Blue" radius="${base_radius}" length="${(base_length - 2*base_radius - enclosure_length)/2}"
@@ -68,36 +57,20 @@
   </link>
   <!-- Handle -->
-  <joint name="handle_joint" type="fixed">
-    <parent link="${tf_prefix}base_link" />
-    <child link="${tf_prefix}handle_link" />
-    <origin xyz="0 0 ${base_radius + handle_height/2}" rpy="0 0 0" />
-  </joint>
+  <xacro:fixed_joint name="handle" xyz="0 0 ${base_radius + handle_height/2}" />
   <link name="${tf_prefix}handle_link">
     <xacro:box_shape color="White" x="${handle_length}" y="${handle_width}" z="${handle_height}" />
   </link>
   <!-- Tray -->
-  <joint name="tray_joint" type="fixed">
-    <parent link="${tf_prefix}base_link" />
-    <child link="${tf_prefix}tray_link" />
-    <origin xyz="0 0 ${-(base_radius + tray_height/2)}" rpy="0 0 0" />
-  </joint>
+  <xacro:fixed_joint name="tray" xyz="0 0 ${-(base_radius + tray_height/2)}" />
   <link name="${tf_prefix}tray_link">
     <xacro:box_shape color="White" x="${tray_length}" y="${tray_width}" z="${tray_height}" />
   </link>
   <!-- Hull -->
-  <joint name="hull_joint" type="fixed">
-    <parent link="${tf_prefix}base_link" />
-    <child link="${tf_prefix}hull_link" />
-    <origin xyz="${(base_length-2*base_radius)/2} 0 0" rpy="0 0 0" />
-  </joint>
+  <xacro:fixed_joint name="hull" xyz="${(base_length-2*base_radius)/2} 0 0" />
   <link name="${tf_prefix}hull_link">
     <xacro:sphere_shape color="Blue" radius="${base_radius}" />
   </link>
   <!-- Thruster -->
-  <joint name="thruster_joint" type="fixed">
-    <parent link="${tf_prefix}base_link" />
-    <child link="${tf_prefix}thruster_link" />
-    <origin xyz="${-(base_length-2*base_radius)/2} 0 0" rpy="0 0 0" />
-  </joint>
+  <xacro:fixed_joint name="thruster" xyz="${-(base_length-2*base_radius)/2} 0 0" />
   <link name="${tf_prefix}thruster_link">
     <xacro:cylinder_shape color="Gray" radius="${base_radius*0.9}" length="${2*base_radius}"

File: coug_description/urdf/rover.urdf.xacro (robot description, xacro)
@@ -71,9 +71,5 @@
   <xacro:wheel prefix="rear_right" xoff="${-wheel_xoff}" y_reflect="-1" />
   <!-- Mast -->
-  <joint name="mast_joint" type="fixed">
-    <parent link="${tf_prefix}base_link" />
-    <child link="${tf_prefix}mast_link" />
-    <origin xyz="${base_length/2 + mast_length/2} 0 ${mast_height/2 - base_height/2}" rpy="0 0 0" />
-  </joint>
+  <xacro:fixed_joint name="mast" xyz="${base_length/2 + mast_length/2} 0 ${mast_height/2 - base_height/2}" />
   <link name="${tf_prefix}mast_link">
     <xacro:box_shape color="LightGray" x="${mast_length}" y="${mast_width}" z="${mast_height}"

File: coug_description/urdf/sensors.gazebo.xacro (robot description, xacro)
@@ -13,6 +13,6 @@
 -->
 <robot xmlns:xacro="http://www.ros.org/wiki/xacro">
-  <xacro:macro name="add_xyz_noise" params="stddev">
-    <xacro:macro name="add_axis_noise">
+  <xacro:macro name="xyz_noise" params="stddev">
+    <xacro:macro name="axis_noise">
       <noise type="gaussian">
         <mean>0.0</mean>
@@ -21,11 +21,11 @@
     </xacro:macro>
     <x>
-      <xacro:add_axis_noise />
+      <xacro:axis_noise />
     </x>
     <y>
-      <xacro:add_axis_noise />
+      <xacro:axis_noise />
     </y>
     <z>
-      <xacro:add_axis_noise />
+      <xacro:axis_noise />
     </z>
   </xacro:macro>
@@ -68,8 +68,8 @@
             https://github.com/stereolabs/zed-ros2-wrapper/blob/v5.4.1/zed_wrapper/config/common_stereo.yaml -->
           <angular_velocity>
-            <xacro:add_xyz_noise stddev="1.2e-3" />
+            <xacro:xyz_noise stddev="1.2e-3" />
           </angular_velocity>
           <linear_acceleration>
-            <xacro:add_xyz_noise stddev="1.6e-2" />
+            <xacro:xyz_noise stddev="1.6e-2" />
           </linear_acceleration>
         </imu>
@@ -82,5 +82,5 @@
         <magnetometer>
           <!-- https://support.sbg-systems.com/sc/el/latest/ellipse-documentation/hardware-documentation/aiding-sensors -->
-          <xacro:add_xyz_noise stddev="3.0e-7" />
+          <xacro:xyz_noise stddev="3.0e-7" />
         </magnetometer>
       </sensor>

Commit message: XML updates

File: coug_description/urdf/bluerov2_body.xacro (robot description, xacro)
@@ -32,19 +32,11 @@
     </link>
   </xacro:macro>
-  <xacro:thruster prefix="thruster1" xyz="0.14 -0.092 0.0" rpy="${radians(-90)} ${radians(90)} ${radians(-45)}"
-    mesh="t200_ccw_prop.dae" mesh_rpy="${radians(-90)} 0 0" />
-  <xacro:thruster prefix="thruster2" xyz="0.14 0.092 0.0" rpy="${radians(-90)} ${radians(90)} ${radians(-135)}"
-    mesh="t200_ccw_prop.dae" mesh_rpy="${radians(-90)} 0 0" />
-  <xacro:thruster prefix="thruster3" xyz="-0.14 -0.092 0.0" rpy="${radians(-90)} ${radians(90)} ${radians(45)}"
-    mesh="t200_cw_prop.dae" mesh_rpy="${radians(90)} 0 0" />
-  <xacro:thruster prefix="thruster4" xyz="-0.14 0.092 0.0" rpy="${radians(-90)} ${radians(90)} ${radians(135)}"
-    mesh="t200_cw_prop.dae" mesh_rpy="${radians(90)} 0 0" />
-  <xacro:thruster prefix="thruster5" xyz="0.118 -0.215 0.064" rpy="0 0 0"
-    mesh="t200_ccw_prop.dae" mesh_rpy="${radians(-90)} 0 ${radians(90)}" />
-  <xacro:thruster prefix="thruster6" xyz="0.118 0.215 0.064" rpy="0 0 0"
-    mesh="t200_cw_prop.dae" mesh_rpy="${radians(90)} 0 ${radians(90)}" />
-  <xacro:thruster prefix="thruster7" xyz="-0.118 -0.215 0.064" rpy="0 0 0"
-    mesh="t200_cw_prop.dae" mesh_rpy="${radians(90)} 0 ${radians(90)}" />
-  <xacro:thruster prefix="thruster8" xyz="-0.118 0.215 0.064" rpy="0 0 0"
-    mesh="t200_ccw_prop.dae" mesh_rpy="${radians(-90)} 0 ${radians(90)}" />
+  <xacro:thruster prefix="thruster1" xyz="0.14 -0.092 0.0" rpy="${radians(-90)} ${radians(90)} ${radians(-45)}" mesh="t200_ccw_prop.dae" mesh_rpy="${radians(-90)} 0 0" />
+  <xacro:thruster prefix="thruster2" xyz="0.14 0.092 0.0" rpy="${radians(-90)} ${radians(90)} ${radians(-135)}" mesh="t200_ccw_prop.dae" mesh_rpy="${radians(-90)} 0 0" />
+  <xacro:thruster prefix="thruster3" xyz="-0.14 -0.092 0.0" rpy="${radians(-90)} ${radians(90)} ${radians(45)}" mesh="t200_cw_prop.dae" mesh_rpy="${radians(90)} 0 0" />
+  <xacro:thruster prefix="thruster4" xyz="-0.14 0.092 0.0" rpy="${radians(-90)} ${radians(90)} ${radians(135)}" mesh="t200_cw_prop.dae" mesh_rpy="${radians(90)} 0 0" />
+  <xacro:thruster prefix="thruster5" xyz="0.118 -0.215 0.064" rpy="0 0 0" mesh="t200_ccw_prop.dae" mesh_rpy="${radians(-90)} 0 ${radians(90)}" />
+  <xacro:thruster prefix="thruster6" xyz="0.118 0.215 0.064" rpy="0 0 0" mesh="t200_cw_prop.dae" mesh_rpy="${radians(90)} 0 ${radians(90)}" />
+  <xacro:thruster prefix="thruster7" xyz="-0.118 -0.215 0.064" rpy="0 0 0" mesh="t200_cw_prop.dae" mesh_rpy="${radians(90)} 0 ${radians(90)}" />
+  <xacro:thruster prefix="thruster8" xyz="-0.118 0.215 0.064" rpy="0 0 0" mesh="t200_ccw_prop.dae" mesh_rpy="${radians(-90)} 0 ${radians(90)}" />
 </robot>

File: coug_description/urdf/common.xacro (robot description, xacro)
@@ -53,6 +53,5 @@
         <origin xyz="${xyz}" rpy="${rpy}" />
         <mass value="${mass}" />
-        <inertia ixx="${mass*(3*radius*radius + length*length)/12}" ixy="0" ixz="0"
-          iyy="${mass*(3*radius*radius + length*length)/12}" iyz="0" izz="${mass*radius*radius/2}" />
+        <inertia ixx="${mass*(3*radius*radius + length*length)/12}" ixy="0" ixz="0" iyy="${mass*(3*radius*radius + length*length)/12}" iyz="0" izz="${mass*radius*radius/2}" />
       </inertial>
     </xacro:if>
@@ -92,6 +91,5 @@
   </xacro:macro>
   <xacro:macro name="optical_frame" params="name">
-    <xacro:sensor_frame name="${name}_optical" parent="${name}"
-      rpy="${radians(-90)} 0 ${radians(-90)}" />
+    <xacro:sensor_frame name="${name}_optical" parent="${name}" rpy="${radians(-90)} 0 ${radians(-90)}" />
   </xacro:macro>
   <xacro:macro name="dvl_beams" params="layout">

File: coug_description/urdf/couguv_body.xacro (robot description, xacro)
@@ -43,16 +43,13 @@
   <xacro:fixed_joint name="clear_body" />
   <link name="${tf_prefix}clear_body_link">
-    <xacro:cylinder_shape color="Acrylic" radius="${base_radius}" length="${enclosure_length}"
-      rpy="0 ${radians(90)} 0" />
+    <xacro:cylinder_shape color="Acrylic" radius="${base_radius}" length="${enclosure_length}" rpy="0 ${radians(90)} 0" />
   </link>
   <xacro:fixed_joint name="front_body" xyz="${(base_length - 2*base_radius - enclosure_length)/4 + enclosure_length/2} 0 0" />
   <link name="${tf_prefix}front_body_link">
-    <xacro:cylinder_shape color="Blue" radius="${base_radius}" length="${(base_length - 2*base_radius - enclosure_length)/2}"
-      rpy="0 ${radians(90)} 0" />
+    <xacro:cylinder_shape color="Blue" radius="${base_radius}" length="${(base_length - 2*base_radius - enclosure_length)/2}" rpy="0 ${radians(90)} 0" />
   </link>
   <xacro:fixed_joint name="back_body" xyz="${-((base_length - 2*base_radius - enclosure_length)/4 + enclosure_length/2)} 0 0" />
   <link name="${tf_prefix}back_body_link">
-    <xacro:cylinder_shape color="Blue" radius="${base_radius}" length="${(base_length - 2*base_radius - enclosure_length)/2}"
-      rpy="0 ${radians(90)} 0" />
+    <xacro:cylinder_shape color="Blue" radius="${base_radius}" length="${(base_length - 2*base_radius - enclosure_length)/2}" rpy="0 ${radians(90)} 0" />
   </link>
   <!-- Handle -->
@@ -74,6 +71,5 @@
   <xacro:fixed_joint name="thruster" xyz="${-(base_length-2*base_radius)/2} 0 0" />
   <link name="${tf_prefix}thruster_link">
-    <xacro:cylinder_shape color="Gray" radius="${base_radius*0.9}" length="${2*base_radius}"
-      rpy="0 ${radians(90)} 0" />
+    <xacro:cylinder_shape color="Gray" radius="${base_radius*0.9}" length="${2*base_radius}" rpy="0 ${radians(90)} 0" />
   </link>
   <!-- Fins -->
@@ -87,6 +83,5 @@
     </joint>
     <link name="${tf_prefix}${prefix}_fin_link">
-      <xacro:box_shape color="White" x="${fin_length}" y="${fin_width}" z="${fin_height}"
-        xyz="${-fin_length/2} 0 ${base_radius+fin_height/2}" />
+      <xacro:box_shape color="White" x="${fin_length}" y="${fin_width}" z="${fin_height}" xyz="${-fin_length/2} 0 ${base_radius+fin_height/2}" />
     </link>
   </xacro:macro>

File: coug_description/urdf/rover.urdf.xacro (robot description, xacro)
@@ -35,6 +35,5 @@
   <xacro:property name="depth_camera_pitch" value="0.1" />
   <!-- Depth camera pose relative to base_link -->
-  <xacro:property name="rover_depth_camera_xyz"
-    value="${base_length/2 + mast_length/2 + depth_camera_xoff} 0 ${mast_height/2 - base_height/2 + depth_camera_zoff}" />
+  <xacro:property name="rover_depth_camera_xyz" value="${base_length/2 + mast_length/2 + depth_camera_xoff} 0 ${mast_height/2 - base_height/2 + depth_camera_zoff}" />
   <xacro:property name="rover_depth_camera_rpy" value="0 ${depth_camera_pitch} 0" />
   <material name="LightGray">
@@ -47,6 +46,5 @@
   <!-- Chassis -->
   <link name="${tf_prefix}base_link">
-    <xacro:box_shape color="LightGray" x="${base_length}" y="${base_width}" z="${base_height}"
-      mass="${base_mass}" />
+    <xacro:box_shape color="LightGray" x="${base_length}" y="${base_width}" z="${base_height}" mass="${base_mass}" />
   </link>
   <!-- Wheels -->
@@ -60,6 +58,5 @@
     </joint>
     <link name="${tf_prefix}${prefix}_wheel_link">
-      <xacro:cylinder_shape color="DarkGray" radius="${wheel_radius}" length="${wheel_width}"
-        rpy="${radians(90)} 0 0" mass="${wheel_mass}" />
+      <xacro:cylinder_shape color="DarkGray" radius="${wheel_radius}" length="${wheel_width}" rpy="${radians(90)} 0 0" mass="${wheel_mass}" />
     </link>
   </xacro:macro>
@@ -73,10 +70,8 @@
   <xacro:fixed_joint name="mast" xyz="${base_length/2 + mast_length/2} 0 ${mast_height/2 - base_height/2}" />
   <link name="${tf_prefix}mast_link">
-    <xacro:box_shape color="LightGray" x="${mast_length}" y="${mast_width}" z="${mast_height}"
-      mass="${mast_mass}" />
+    <xacro:box_shape color="LightGray" x="${mast_length}" y="${mast_width}" z="${mast_height}" mass="${mast_mass}" />
   </link>
   <!-- Sensors -->
-  <xacro:sensor_frame name="depth_camera" parent="mast" xyz="${depth_camera_xoff} 0 ${depth_camera_zoff}"
-    rpy="${rover_depth_camera_rpy}" />
+  <xacro:sensor_frame name="depth_camera" parent="mast" xyz="${depth_camera_xoff} 0 ${depth_camera_zoff}" rpy="${rover_depth_camera_rpy}" />
   <xacro:optical_frame name="depth_camera" />
   <xacro:sensor_frame name="imu" parent="depth_camera" />

Commit message: Add BlueROV2 mesh source

File: coug_description/urdf/bluerov2_body.xacro (robot description, xacro)
@@ -17,5 +17,5 @@
     <visual>
       <geometry>
-        <mesh filename="package://coug_description/urdf/meshes/bluerov2/bluerov2.dae" scale="0.025 0.025 0.025" />
+        <mesh filename="package://blue_description/meshes/bluerov2_heavy/bluerov2_heavy.dae" scale="0.025 0.025 0.025" />
       </geometry>
     </visual>
@@ -27,16 +27,16 @@
         <origin xyz="0 0 0" rpy="${mesh_rpy}" />
         <geometry>
-          <mesh filename="package://coug_description/urdf/meshes/bluerov2/${mesh}" />
+          <mesh filename="package://blue_description/meshes/t200/${mesh}" />
         </geometry>
       </visual>
     </link>
   </xacro:macro>
-  <xacro:thruster prefix="thruster1" xyz="0.14 -0.092 0.0" rpy="${radians(-90)} ${radians(90)} ${radians(-45)}" mesh="t200_ccw_prop.dae" mesh_rpy="${radians(-90)} 0 0" />
-  <xacro:thruster prefix="thruster2" xyz="0.14 0.092 0.0" rpy="${radians(-90)} ${radians(90)} ${radians(-135)}" mesh="t200_ccw_prop.dae" mesh_rpy="${radians(-90)} 0 0" />
-  <xacro:thruster prefix="thruster3" xyz="-0.14 -0.092 0.0" rpy="${radians(-90)} ${radians(90)} ${radians(45)}" mesh="t200_cw_prop.dae" mesh_rpy="${radians(90)} 0 0" />
-  <xacro:thruster prefix="thruster4" xyz="-0.14 0.092 0.0" rpy="${radians(-90)} ${radians(90)} ${radians(135)}" mesh="t200_cw_prop.dae" mesh_rpy="${radians(90)} 0 0" />
-  <xacro:thruster prefix="thruster5" xyz="0.118 -0.215 0.064" rpy="0 0 0" mesh="t200_ccw_prop.dae" mesh_rpy="${radians(-90)} 0 ${radians(90)}" />
-  <xacro:thruster prefix="thruster6" xyz="0.118 0.215 0.064" rpy="0 0 0" mesh="t200_cw_prop.dae" mesh_rpy="${radians(90)} 0 ${radians(90)}" />
-  <xacro:thruster prefix="thruster7" xyz="-0.118 -0.215 0.064" rpy="0 0 0" mesh="t200_cw_prop.dae" mesh_rpy="${radians(90)} 0 ${radians(90)}" />
-  <xacro:thruster prefix="thruster8" xyz="-0.118 0.215 0.064" rpy="0 0 0" mesh="t200_ccw_prop.dae" mesh_rpy="${radians(-90)} 0 ${radians(90)}" />
+  <xacro:thruster prefix="thruster1" xyz="0.14 -0.092 0.0" rpy="${radians(-90)} ${radians(90)} ${radians(-45)}" mesh="ccw_prop.dae" mesh_rpy="${radians(-90)} 0 0" />
+  <xacro:thruster prefix="thruster2" xyz="0.14 0.092 0.0" rpy="${radians(-90)} ${radians(90)} ${radians(-135)}" mesh="ccw_prop.dae" mesh_rpy="${radians(-90)} 0 0" />
+  <xacro:thruster prefix="thruster3" xyz="-0.14 -0.092 0.0" rpy="${radians(-90)} ${radians(90)} ${radians(45)}" mesh="cw_prop.dae" mesh_rpy="${radians(90)} 0 0" />
+  <xacro:thruster prefix="thruster4" xyz="-0.14 0.092 0.0" rpy="${radians(-90)} ${radians(90)} ${radians(135)}" mesh="cw_prop.dae" mesh_rpy="${radians(90)} 0 0" />
+  <xacro:thruster prefix="thruster5" xyz="0.118 -0.215 0.064" rpy="0 0 0" mesh="ccw_prop.dae" mesh_rpy="${radians(-90)} 0 ${radians(90)}" />
+  <xacro:thruster prefix="thruster6" xyz="0.118 0.215 0.064" rpy="0 0 0" mesh="cw_prop.dae" mesh_rpy="${radians(90)} 0 ${radians(90)}" />
+  <xacro:thruster prefix="thruster7" xyz="-0.118 -0.215 0.064" rpy="0 0 0" mesh="cw_prop.dae" mesh_rpy="${radians(90)} 0 ${radians(90)}" />
+  <xacro:thruster prefix="thruster8" xyz="-0.118 0.215 0.064" rpy="0 0 0" mesh="ccw_prop.dae" mesh_rpy="${radians(-90)} 0 ${radians(90)}" />
 </robot>
