Commit message: URDF cleanup

File: coug_description/urdf/blueboat.urdf.xacro (robot description, xacro)
@@ -16,14 +16,16 @@
   <xacro:property name="tf_prefix" value="$(arg tf_prefix)" />
   <xacro:include filename="$(find coug_description)/urdf/common.xacro" />
-  <xacro:property name="base_height" value="0.40" />
+  <!-- https://discuss.bluerobotics.com/t/blueboat-reference-point/23072 -->
+  <xacro:property name="blueboat_mesh_zoff" value="0.188" />
+  <xacro:property name="base_height" value="0.4" />
   <xacro:property name="base_width" value="0.93" />
-  <xacro:property name="base_length" value="1.20" />
+  <xacro:property name="base_length" value="1.2" />
   <!-- 14.5 kg dry + 2x 4S Li-ion batteries + sensor payload -->
   <xacro:property name="base_mass" value="18.0" />
-  <xacro:property name="thruster_xoff" value="-0.488" />
+  <xacro:property name="thruster_xoff" value="0.488" />
   <xacro:property name="thruster_yoff" value="0.295" />
-  <xacro:property name="thruster_zoff" value="-0.272" />
+  <xacro:property name="thruster_zoff" value="${0.272 - blueboat_mesh_zoff}" />
   <xacro:property name="thruster_mass" value="0.2" />
-  <xacro:property name="blueboat_depth_camera_xyz" value="0.45 0 0.15" />
+  <xacro:property name="blueboat_depth_camera_xyz" value="0.45 0 ${blueboat_mesh_zoff + 0.15}" />
   <xacro:property name="blueboat_depth_camera_rpy" value="0 ${radians(10)} 0" />
   <material name="Black">
@@ -36,7 +38,7 @@
     <color rgba="1 1 0 1" />
   </material>
-  <xacro:macro name="mesh_visual" params="mesh color rpy:='0 0 0'">
+  <xacro:macro name="mesh_shape" params="mesh color xyz:='0 0 ${blueboat_mesh_zoff}' rpy:='0 0 0'">
     <visual>
-      <origin xyz="0 0 0" rpy="${rpy}" />
+      <origin xyz="${xyz}" rpy="${rpy}" />
       <geometry>
         <mesh filename="package://ardupilot_sitl_models/models/blueboat/meshes/blueboat_${mesh}.dae" />
@@ -47,36 +49,32 @@
   <!-- Hull -->
   <link name="${tf_prefix}base_link">
-    <xacro:mesh_visual mesh="hull" color="Blue" />
-    <xacro:mesh_visual mesh="aerial" color="Black" />
-    <xacro:mesh_visual mesh="crosstube" color="Black" />
-    <xacro:mesh_visual mesh="flag" color="Yellow" />
-    <xacro:mesh_visual mesh="frame_asm_aft" color="Black" />
-    <xacro:mesh_visual mesh="frame_asm_fore" color="Black" />
-    <xacro:mesh_visual mesh="hatch_asm_port" color="Black" />
-    <xacro:mesh_visual mesh="hatch_asm_stbd" color="Black" />
-    <xacro:mesh_visual mesh="motor_port" color="Black" />
-    <xacro:mesh_visual mesh="motor_stbd" color="Black" />
+    <xacro:mesh_shape mesh="hull" color="Blue" />
+    <xacro:mesh_shape mesh="aerial" color="Black" />
+    <xacro:mesh_shape mesh="crosstube" color="Black" />
+    <xacro:mesh_shape mesh="flag" color="Yellow" />
+    <xacro:mesh_shape mesh="frame_asm_aft" color="Black" />
+    <xacro:mesh_shape mesh="frame_asm_fore" color="Black" />
+    <xacro:mesh_shape mesh="hatch_asm_port" color="Black" />
+    <xacro:mesh_shape mesh="hatch_asm_stbd" color="Black" />
+    <xacro:mesh_shape mesh="motor_port" color="Black" />
+    <xacro:mesh_shape mesh="motor_stbd" color="Black" />
     <collision>
+      <origin xyz="0 0 ${blueboat_mesh_zoff}" />
       <geometry>
         <mesh filename="package://ardupilot_sitl_models/models/blueboat/meshes/blueboat_hull_collision.stl" />
       </geometry>
     </collision>
-    <inertial>
-      <origin xyz="-0.05 0 -0.15" />
-      <mass value="${base_mass}" />
-      <inertia ixx="${base_mass*(base_width*base_width + base_height*base_height)/12}" ixy="0" ixz="0" iyy="${base_mass*(base_length*base_length + base_height*base_height)/12}" iyz="0" izz="${base_mass*(base_length*base_length + base_width*base_width)/12}" />
-    </inertial>
+    <xacro:box_inertial x="${base_length}" y="${base_width}" z="${base_height}" mass="${base_mass}" />
   </link>
   <!-- Thrusters -->
-  <xacro:macro name="thruster" params="prefix y_reflect mesh">
+  <xacro:macro name="thruster" params="prefix y_reflect">
     <joint name="${prefix}_thruster_joint" type="continuous">
       <parent link="${tf_prefix}base_link" />
       <child link="${tf_prefix}${prefix}_thruster_link" />
-      <origin xyz="${thruster_xoff} ${y_reflect*thruster_yoff} ${thruster_zoff}" rpy="0 0 0" />
+      <origin xyz="${-thruster_xoff} ${y_reflect*thruster_yoff} ${-thruster_zoff}" rpy="0 0 0" />
       <axis xyz="1 0 0" />
-      <dynamics damping="0.02" />
     </joint>
     <link name="${tf_prefix}${prefix}_thruster_link">
-      <xacro:mesh_visual mesh="${mesh}" color="Black" rpy="${radians(-90)} 0 ${radians(90)}" />
+      <xacro:mesh_shape mesh="prop_${'port' if y_reflect == 1 else 'stbd'}" color="Black" xyz="0 0 0" rpy="${radians(-90)} 0 ${radians(90)}" />
       <inertial>
         <mass value="${thruster_mass}" />
@@ -85,9 +83,9 @@
     </link>
   </xacro:macro>
-  <xacro:thruster prefix="left" y_reflect="1" mesh="prop_port" />
-  <xacro:thruster prefix="right" y_reflect="-1" mesh="prop_stbd" />
+  <xacro:thruster prefix="left" y_reflect="1" />
+  <xacro:thruster prefix="right" y_reflect="-1" />
   <!-- Sensors -->
-  <xacro:sensor_frame name="gps" xyz="0.16 -0.365 0.03" />
-  <xacro:sensor_frame name="imu" xyz="0.16 -0.365 -0.07" />
+  <xacro:sensor_frame name="imu" xyz="0.16 -0.365 0.12" />
+  <xacro:sensor_frame name="gps" xyz="0.16 -0.365 0.22" />
   <xacro:sensor_frame name="depth_camera" xyz="${blueboat_depth_camera_xyz}" rpy="${blueboat_depth_camera_rpy}" />
   <xacro:optical_frame name="depth_camera" />

File: coug_description/urdf/bluerov2_body.xacro (robot description, xacro)
@@ -13,4 +13,5 @@
 -->
 <robot xmlns:xacro="http://www.ros.org/wiki/xacro">
+  <!-- Body -->
   <link name="${tf_prefix}base_link">
     <visual>
@@ -20,4 +21,5 @@
     </visual>
   </link>
+  <!-- Thrusters -->
   <xacro:macro name="thruster" params="prefix xyz rpy mesh mesh_rpy">
     <xacro:fixed_joint name="${prefix}" xyz="${xyz}" rpy="${rpy}" />
@@ -31,8 +33,8 @@
     </link>
   </xacro:macro>
-  <xacro:thruster prefix="thruster1" xyz="0.14 -0.092 0.0" rpy="${radians(-90)} ${radians(90)} ${radians(-45)}" mesh="ccw_prop.dae" mesh_rpy="${radians(-90)} 0 0" />
-  <xacro:thruster prefix="thruster2" xyz="0.14 0.092 0.0" rpy="${radians(-90)} ${radians(90)} ${radians(-135)}" mesh="ccw_prop.dae" mesh_rpy="${radians(-90)} 0 0" />
-  <xacro:thruster prefix="thruster3" xyz="-0.14 -0.092 0.0" rpy="${radians(-90)} ${radians(90)} ${radians(45)}" mesh="cw_prop.dae" mesh_rpy="${radians(90)} 0 0" />
-  <xacro:thruster prefix="thruster4" xyz="-0.14 0.092 0.0" rpy="${radians(-90)} ${radians(90)} ${radians(135)}" mesh="cw_prop.dae" mesh_rpy="${radians(90)} 0 0" />
+  <xacro:thruster prefix="thruster1" xyz="0.14 -0.092 0" rpy="${radians(-90)} ${radians(90)} ${radians(-45)}" mesh="ccw_prop.dae" mesh_rpy="${radians(-90)} 0 0" />
+  <xacro:thruster prefix="thruster2" xyz="0.14 0.092 0" rpy="${radians(-90)} ${radians(90)} ${radians(-135)}" mesh="ccw_prop.dae" mesh_rpy="${radians(-90)} 0 0" />
+  <xacro:thruster prefix="thruster3" xyz="-0.14 -0.092 0" rpy="${radians(-90)} ${radians(90)} ${radians(45)}" mesh="cw_prop.dae" mesh_rpy="${radians(90)} 0 0" />
+  <xacro:thruster prefix="thruster4" xyz="-0.14 0.092 0" rpy="${radians(-90)} ${radians(90)} ${radians(135)}" mesh="cw_prop.dae" mesh_rpy="${radians(90)} 0 0" />
   <xacro:thruster prefix="thruster5" xyz="0.118 -0.215 0.064" rpy="0 0 0" mesh="ccw_prop.dae" mesh_rpy="${radians(-90)} 0 ${radians(90)}" />
   <xacro:thruster prefix="thruster6" xyz="0.118 0.215 0.064" rpy="0 0 0" mesh="cw_prop.dae" mesh_rpy="${radians(90)} 0 ${radians(90)}" />

File: coug_description/urdf/common.xacro (robot description, xacro)
@@ -13,4 +13,11 @@
 -->
 <robot xmlns:xacro="http://www.ros.org/wiki/xacro">
+  <xacro:macro name="box_inertial" params="x y z mass xyz:='0 0 0' rpy:='0 0 0'">
+    <inertial>
+      <origin xyz="${xyz}" rpy="${rpy}" />
+      <mass value="${mass}" />
+      <inertia ixx="${mass*(y*y + z*z)/12}" ixy="0" ixz="0" iyy="${mass*(x*x + z*z)/12}" iyz="0" izz="${mass*(x*x + y*y)/12}" />
+    </inertial>
+  </xacro:macro>
   <xacro:macro name="box_shape" params="color x y z xyz:='0 0 0' rpy:='0 0 0' mass:=0">
     <visual>
@@ -28,9 +35,5 @@
         </geometry>
       </collision>
-      <inertial>
-        <origin xyz="${xyz}" rpy="${rpy}" />
-        <mass value="${mass}" />
-        <inertia ixx="${mass*(y*y + z*z)/12}" ixy="0" ixz="0" iyy="${mass*(x*x + z*z)/12}" iyz="0" izz="${mass*(x*x + y*y)/12}" />
-      </inertial>
+      <xacro:box_inertial x="${x}" y="${y}" z="${z}" mass="${mass}" xyz="${xyz}" rpy="${rpy}" />
     </xacro:if>
   </xacro:macro>

File: coug_description/urdf/couguv_body.xacro (robot description, xacro)
@@ -16,4 +16,5 @@
   <xacro:property name="base_length" value="1.2" />
   <xacro:property name="enclosure_length" value="0.5" />
+  <xacro:property name="body_length" value="${(base_length - 2*base_radius - enclosure_length)/2}" />
   <xacro:property name="handle_height" value="0.07" />
   <xacro:property name="handle_width" value="0.04" />
@@ -22,8 +23,8 @@
   <xacro:property name="tray_width" value="0.05" />
   <xacro:property name="tray_length" value="0.38" />
-  <xacro:property name="fin_xoff" value="0.375" />
   <xacro:property name="fin_height" value="0.09" />
   <xacro:property name="fin_width" value="0.015" />
   <xacro:property name="fin_length" value="0.09" />
+  <xacro:property name="fin_xoff" value="0.375" />
   <material name="White">
     <color rgba="1 1 1 1" />
@@ -44,11 +45,11 @@
     <xacro:cylinder_shape color="Acrylic" radius="${base_radius}" length="${enclosure_length}" rpy="0 ${radians(90)} 0" />
   </link>
-  <xacro:fixed_joint name="front_body" xyz="${(base_length - 2*base_radius - enclosure_length)/4 + enclosure_length/2} 0 0" />
+  <xacro:fixed_joint name="front_body" xyz="${body_length/2 + enclosure_length/2} 0 0" />
   <link name="${tf_prefix}front_body_link">
-    <xacro:cylinder_shape color="Blue" radius="${base_radius}" length="${(base_length - 2*base_radius - enclosure_length)/2}" rpy="0 ${radians(90)} 0" />
+    <xacro:cylinder_shape color="Blue" radius="${base_radius}" length="${body_length}" rpy="0 ${radians(90)} 0" />
   </link>
-  <xacro:fixed_joint name="back_body" xyz="${-((base_length - 2*base_radius - enclosure_length)/4 + enclosure_length/2)} 0 0" />
+  <xacro:fixed_joint name="back_body" xyz="${-(body_length/2 + enclosure_length/2)} 0 0" />
   <link name="${tf_prefix}back_body_link">
-    <xacro:cylinder_shape color="Blue" radius="${base_radius}" length="${(base_length - 2*base_radius - enclosure_length)/2}" rpy="0 ${radians(90)} 0" />
+    <xacro:cylinder_shape color="Blue" radius="${base_radius}" length="${body_length}" rpy="0 ${radians(90)} 0" />
   </link>
   <!-- Handle -->
@@ -63,10 +64,10 @@
   </link>
   <!-- Hull -->
-  <xacro:fixed_joint name="hull" xyz="${(base_length-2*base_radius)/2} 0 0" />
+  <xacro:fixed_joint name="hull" xyz="${base_length/2 - base_radius} 0 0" />
   <link name="${tf_prefix}hull_link">
     <xacro:sphere_shape color="Blue" radius="${base_radius}" />
   </link>
   <!-- Thruster -->
-  <xacro:fixed_joint name="thruster" xyz="${-(base_length-2*base_radius)/2} 0 0" />
+  <xacro:fixed_joint name="thruster" xyz="${-(base_length/2 - base_radius)} 0 0" />
   <link name="${tf_prefix}thruster_link">
     <xacro:cylinder_shape color="Gray" radius="${base_radius*0.9}" length="${2*base_radius}" rpy="0 ${radians(90)} 0" />
@@ -82,5 +83,5 @@
     </joint>
     <link name="${tf_prefix}${prefix}_fin_link">
-      <xacro:box_shape color="White" x="${fin_length}" y="${fin_width}" z="${fin_height}" xyz="${-fin_length/2} 0 ${base_radius+fin_height/2}" />
+      <xacro:box_shape color="White" x="${fin_length}" y="${fin_width}" z="${fin_height}" xyz="${-fin_length/2} 0 ${base_radius + fin_height/2}" />
     </link>
   </xacro:macro>

File: coug_description/urdf/rover.urdf.xacro (robot description, xacro)
@@ -19,8 +19,8 @@
   <xacro:property name="base_width" value="0.5" />
   <xacro:property name="base_length" value="0.4" />
-  <xacro:property name="base_xoff" value="0.135" />
   <xacro:property name="base_mass" value="18.0" />
   <xacro:property name="wheel_radius" value="0.15" />
   <xacro:property name="wheel_width" value="0.2" />
+  <xacro:property name="middle_wheel_xoff" value="0.135" />
   <xacro:property name="wheel_xoff" value="0.7" />
   <xacro:property name="wheel_yoff" value="${base_width/2 + 0.1 + wheel_width/2}" />
@@ -33,5 +33,5 @@
   <xacro:property name="depth_camera_xoff" value="0.12" />
   <xacro:property name="depth_camera_zoff" value="0.05" />
-  <xacro:property name="depth_camera_pitch" value="0.1" />
+  <xacro:property name="depth_camera_pitch" value="${radians(6)}" />
   <xacro:property name="rover_depth_camera_xyz" value="${base_length/2 + mast_length/2 + depth_camera_xoff} 0 ${mast_height/2 - base_height/2 + depth_camera_zoff}" />
   <xacro:property name="rover_depth_camera_rpy" value="0 ${depth_camera_pitch} 0" />
@@ -52,5 +52,5 @@
       <parent link="${tf_prefix}base_link" />
       <child link="${tf_prefix}${prefix}_wheel_link" />
-      <origin xyz="${base_xoff + xoff} ${y_reflect*wheel_yoff} ${-wheel_zoff}" rpy="0 0 0" />
+      <origin xyz="${middle_wheel_xoff + xoff} ${y_reflect*wheel_yoff} ${-wheel_zoff}" rpy="0 0 0" />
       <axis xyz="0 1 0" />
       <dynamics damping="0.05" friction="0.1" />

Commit message: Add BlueBoat links

File: coug_description/urdf/blueboat.urdf.xacro (robot description, xacro)
@@ -18,9 +18,13 @@
   <!-- https://discuss.bluerobotics.com/t/blueboat-reference-point/23072 -->
   <xacro:property name="blueboat_mesh_zoff" value="0.188" />
-  <xacro:property name="base_height" value="0.4" />
+  <!-- https://bluerobotics.com/store/boat/blueboat/blueboat/ -->
+  <xacro:property name="base_height" value="0.46" />
   <xacro:property name="base_width" value="0.93" />
   <xacro:property name="base_length" value="1.2" />
-  <!-- 14.5 kg dry + 2x 4S Li-ion batteries + sensor payload -->
+  <!-- 14.5 kg dry + 2x 1.163 kg batteries + ~1.2 kg payload
+    https://bluerobotics.com/store/boat/blueboat/blueboat/
+    https://bluerobotics.com/store/comm-control-power/powersupplies-batteries/battery-li-4s-15-6ah/ -->
   <xacro:property name="base_mass" value="18.0" />
+  <!-- https://github.com/ArduPilot/SITL_Models/blob/master/Gazebo/models/blueboat/model.sdf -->
   <xacro:property name="thruster_xoff" value="0.488" />
   <xacro:property name="thruster_yoff" value="0.295" />
@@ -86,4 +90,5 @@
   <xacro:thruster prefix="right" y_reflect="-1" />
   <!-- Sensors -->
+  <!-- https://github.com/bluerobotics/Blueos-Parameter-Repository/blob/master/params/ardupilot/ArduRover/4.7/Navigator/BlueBoat120.params -->
   <xacro:sensor_frame name="imu" xyz="0.16 -0.365 0.12" />
   <xacro:sensor_frame name="gps" xyz="0.16 -0.365 0.22" />

Commit message: Better Blueboat params

File: coug_description/urdf/blueboat.urdf.xacro (robot description, xacro)
@@ -22,8 +22,9 @@
   <xacro:property name="base_width" value="0.93" />
   <xacro:property name="base_length" value="1.2" />
-  <!-- 14.5 kg dry + 2x 1.163 kg batteries + ~1.2 kg payload
-    https://bluerobotics.com/store/boat/blueboat/blueboat/
+  <!-- https://bluerobotics.com/store/boat/blueboat/blueboat/
     https://bluerobotics.com/store/comm-control-power/powersupplies-batteries/battery-li-4s-15-6ah/ -->
-  <xacro:property name="base_mass" value="18.0" />
+  <xacro:property name="base_mass" value="${14.5 + 2*1.163 - 2*thruster_mass}" />
+  <!-- https://bluerobotics.com/store/boat/blueboat/blueboat/ -->
+  <xacro:property name="thruster_radius" value="${0.112/2}" />
   <!-- https://github.com/ArduPilot/SITL_Models/blob/master/Gazebo/models/blueboat/model.sdf -->
   <xacro:property name="thruster_xoff" value="0.488" />
@@ -81,8 +82,5 @@
     <link name="${tf_prefix}${prefix}_thruster_link">
       <xacro:mesh_shape mesh="prop_${'port' if y_reflect == 1 else 'stbd'}" color="Black" xyz="0 0 0" rpy="${radians(-90)} 0 ${radians(90)}" />
-      <inertial>
-        <mass value="${thruster_mass}" />
-        <inertia ixx="0.0001" ixy="0" ixz="0" iyy="0.0001" iyz="0" izz="0.0001" />
-      </inertial>
+      <xacro:cylinder_inertial radius="${thruster_radius}" length="0" mass="${thruster_mass}" rpy="0 ${radians(90)} 0" />
     </link>
   </xacro:macro>

File: coug_description/urdf/common.xacro (robot description, xacro)
@@ -38,4 +38,11 @@
     </xacro:if>
   </xacro:macro>
+  <xacro:macro name="cylinder_inertial" params="radius length mass xyz:='0 0 0' rpy:='0 0 0'">
+    <inertial>
+      <origin xyz="${xyz}" rpy="${rpy}" />
+      <mass value="${mass}" />
+      <inertia ixx="${mass*(3*radius*radius + length*length)/12}" ixy="0" ixz="0" iyy="${mass*(3*radius*radius + length*length)/12}" iyz="0" izz="${mass*radius*radius/2}" />
+    </inertial>
+  </xacro:macro>
   <xacro:macro name="cylinder_shape" params="color radius length xyz:='0 0 0' rpy:='0 0 0' mass:=0">
     <visual>
@@ -53,9 +60,5 @@
         </geometry>
       </collision>
-      <inertial>
-        <origin xyz="${xyz}" rpy="${rpy}" />
-        <mass value="${mass}" />
-        <inertia ixx="${mass*(3*radius*radius + length*length)/12}" ixy="0" ixz="0" iyy="${mass*(3*radius*radius + length*length)/12}" iyz="0" izz="${mass*radius*radius/2}" />
-      </inertial>
+      <xacro:cylinder_inertial radius="${radius}" length="${length}" mass="${mass}" xyz="${xyz}" rpy="${rpy}" />
     </xacro:if>
   </xacro:macro>
