Commit message: Better TURTLMap URDF

File: coug_description/urdf/turtlmap.urdf.xacro (robot description, xacro)
@@ -37,5 +37,5 @@
     <parent link="base_link"/>
     <child link="dvl_link"/>
-    <origin xyz="0.11247 0.00146 -0.04147" rpy="${pi} 0 0"/>
+    <origin xyz="0.113 0.001 -0.04" rpy="${pi} 0 0"/>
   </joint>
 </robot>

Commit message: Fixed TURTLMap ZED frame

File: coug_description/urdf/turtlmap.urdf.xacro (robot description, xacro)
@@ -82,7 +82,7 @@
   <!-- ZED Mini Camera Link -->
   <joint name="zedm_left_camera_joint" type="fixed">
-    <parent link="imu_link" />
+    <parent link="base_link" />
     <child link="zedm_left_camera_frame" />
-    <origin xyz="0 0 0" rpy="0 0 0" />
+    <origin xyz="0 0 0" rpy="${-pi/2} ${pi/2} 0" />
   </joint>
   <link name="zedm_left_camera_frame" />

Commit message: Add depth cam offset

File: coug_description/urdf/turtlmap.urdf.xacro (robot description, xacro)
@@ -27,5 +27,5 @@
     <parent link="${tf_prefix}base_link" />
     <child link="${tf_prefix}zedm_left_camera_frame" />
-    <origin xyz="0 0 0" rpy="${radians(-90)} ${radians(90)} 0" />
+    <origin xyz="0.212 0.0652 0.006" rpy="${radians(-90)} ${radians(90)} 0" />
   </joint>
   <link name="${tf_prefix}zedm_left_camera_frame" />

Commit message: Revert turtlmap bug

File: coug_description/urdf/turtlmap.urdf.xacro (robot description, xacro)
@@ -27,5 +27,5 @@
     <parent link="${tf_prefix}base_link" />
     <child link="${tf_prefix}zedm_left_camera_frame" />
-    <origin xyz="0.212 0.0652 0.006" rpy="${radians(-90)} ${radians(90)} 0" />
+    <origin xyz="0 0 0" rpy="${radians(-90)} ${radians(90)} 0" />
   </joint>
   <link name="${tf_prefix}zedm_left_camera_frame" />
